Commit message: reduced urdf file size

File: src/subjugator/simulation/urdf/sub9.urdf.xacro (robot description, xacro)
@@ -16,5 +16,5 @@
       <origin rpy="${pi/2} 0 ${pi}" xyz="${(0.915/2-0.009)} ${-(0.606/2)} ${-(0.381/2)}"/>
       <geometry>
-        <mesh filename="./meshes/Sub9"/>
+        <mesh filename="./meshes/sub9.dae"/>
       </geometry>
     </visual>
@@ -22,5 +22,5 @@
       <origin rpy="${pi/2} 0 ${pi}" xyz="${(0.915/2-0.009)} ${-(0.606/2)} ${-(0.381/2)}"/>
       <geometry>
-        <mesh filename="./meshes/Sub9"/>
+        <mesh filename="./meshes/sub9.dae"/>
       </geometry>
     </collision>
