Commit message: Trying to figure out why Plugin Configure is not being run

File: src/subjugator/simulation/subjugator_description/urdf/xacro/hydrophone.xacro (robot description, xacro)
@@ -2,10 +2,7 @@
 <robot xmlns:xacro="http://ros.org/wiki/xacro" xmlns:experimental="http://sdformat.org/schemas/experimental" xmlns:gz="http://gazebosim.org/schema">
   <!-- Macro for inserting a Hydrophone -->
-  <xacro:macro
-    name="mil_hydrophone"
-    params="name parent xyz rpy"
-  >
+  <xacro:macro name="mil_hydrophone" params="name parent xyz rpy">
     <!-- Hydrophone Link -->
-     <link name="${name}_link">
+    <link name="${name}_link">
       <origin xyz="0 0 0" rpy="0 0 0"/>
       <inertial>
@@ -27,9 +24,7 @@
     </gazebo>
     <gazebo reference="${name}_link">
-      <plugin
-            filename="Hydrophone"
-            name="hydrophone::Hydrophone">
-            <topic>${name}</topic>
-        </plugin>
+      <plugin filename="DVLBridge" name="dave_ros_gz_plugins::DVLBridge">
+        <topic>${name}</topic>
+      </plugin>
     </gazebo>
   </xacro:macro>
