Commit message: The gripper arms open and close on keyboard press! Now I need to test if they can pick up objects

File: src/subjugator/simulation/subjugator_description/urdf/xacro/gripper.xacro (robot description, xacro)
@@ -37,11 +37,5 @@
         </geometry>
       </visual>
-      <!-- Left Arm Collision -->
-      <!-- <collision>
-        <origin xyz="0 0.025 -0.3" rpy="1.57 0 -1.57"/>
-        <geometry>
-          <mesh filename="package://subjugator_description/models/gripper_2025/gripper_arm.dae"/>
-        </geometry>
-      </collision> -->
+      <!-- Left arm collision removed to avoid crossing/overlap issues during motion -->
     </link>
     <!-- Left Arm Joint -->
@@ -50,5 +44,5 @@
       <parent link="${name}_link"/>
       <child link="${name}_leftArm_link"/>
-      <axis xyz="0 1 0"/>
+      <axis xyz="1 0 0"/>
       <limit effort="1.0" velocity="1.0" lower="0.0" upper="0.5"/>
     </joint>
@@ -67,11 +61,5 @@
         </geometry>
       </visual>
-      <!-- Right Arm Collision -->
-      <!-- <collision>
-        <origin xyz="0 -0.025 -0.3" rpy="1.57 0 1.57"/>
-        <geometry>
-          <mesh filename="package://subjugator_description/models/gripper_2025/gripper_arm.dae"/>
-        </geometry>
-      </collision> -->
+      <!-- Right arm collision removed to avoid crossing/overlap issues during motion -->
     </link>
     <!-- Right Arm Joint -->
@@ -80,5 +68,5 @@
       <parent link="${name}_link"/>
       <child link="${name}_rightArm_link"/>
-      <axis xyz="0 1 0"/>
+      <axis xyz="-1 0 0"/>
       <limit effort="1.0" velocity="1.0" lower="0.0" upper="0.5"/>
     </joint>

Commit message: I moved the collision box down more to hopefully fix but Im leaving before testing those changes (nice)

File: src/subjugator/simulation/subjugator_description/urdf/xacro/gripper.xacro (robot description, xacro)
@@ -39,11 +39,20 @@
       <!-- Left fingertip collision: small rectangular box for reliable contact -->
       <collision name="leftArm_collision">
-        <!-- positioned near the visual fingertip; adjust if needed -->
-        <origin xyz="0 0.045 0" rpy="0 0 0"/>
+        <!-- positioned to align with the visual finger tip (z ~ -0.3) -->
+        <origin xyz="0 0.045 -0.32" rpy="0 0 0"/>
         <geometry>
           <box>
-            <size>0.1 0.1 0.1</size>
+            <size>0.02 0.04 0.06</size>
           </box>
         </geometry>
+        <!-- simple friction hint (Gazebo/ODE) -->
+        <surface>
+          <friction>
+            <ode>
+              <mu>1.0</mu>
+              <mu2>1.0</mu2>
+            </ode>
+          </friction>
+        </surface>
       </collision>
     </link>
@@ -72,11 +81,20 @@
       <!-- Right fingertip collision: small rectangular box for reliable contact -->
       <collision name="rightArm_collision">
-        <!-- positioned near the visual fingertip; adjust if needed -->
-        <origin xyz="0 -0.045 0" rpy="0 0 0"/>
+        <!-- positioned to align with the visual finger tip (z ~ -0.3) -->
+        <origin xyz="0 -0.045 -0.32" rpy="0 0 0"/>
         <geometry>
           <box>
-            <size>0.1 0.1 0.1</size>
+            <size>0.02 0.04 0.06</size>
           </box>
         </geometry>
+        <!-- simple friction hint (Gazebo/ODE) -->
+        <surface>
+          <friction>
+            <ode>
+              <mu>1.0</mu>
+              <mu2>1.0</mu2>
+            </ode>
+          </friction>
+        </surface>
       </collision>
     </link>
