Commit message: Fixed gazebo reset crashing by adding alternate DVL sensor in RL specific subjugator description

File: src/subjugator/Reinforcement_Learning/src/rl_subjugator_description/urdf/sub9.urdf.xacro (robot description, xacro)
@@ -2,12 +2,12 @@
 <robot xmlns:xacro="http://www.ros.org/wiki/xacro" name="sub9">
   <!-- XACRO INCLUDES -->
-  <xacro:include filename="$(find subjugator_description)/urdf/xacro/fixed_link.xacro"/>
-  <xacro:include filename="$(find subjugator_description)/urdf/xacro/camera.xacro"/>
-  <xacro:include filename="$(find subjugator_description)/urdf/xacro/imu_magnetometer.xacro"/>
-  <xacro:include filename="$(find subjugator_description)/urdf/xacro/dvl.xacro"/>
-  <xacro:include filename="$(find subjugator_description)/urdf/xacro/hydrophone.xacro"/>
-  <xacro:include filename="$(find subjugator_description)/urdf/xacro/collision.xacro"/>
-  <xacro:include filename="$(find subjugator_description)/urdf/xacro/thruster.xacro"/>
-  <xacro:include filename="$(find subjugator_description)/urdf/xacro/depth.xacro"/>
+  <xacro:include filename="$(find rl_subjugator_description)/urdf/xacro/fixed_link.xacro"/>
+  <xacro:include filename="$(find rl_subjugator_description)/urdf/xacro/camera.xacro"/>
+  <xacro:include filename="$(find rl_subjugator_description)/urdf/xacro/imu_magnetometer.xacro"/>
+  <xacro:include filename="$(find rl_subjugator_description)/urdf/xacro/dvl.xacro"/>
+  <xacro:include filename="$(find rl_subjugator_description)/urdf/xacro/hydrophone.xacro"/>
+  <xacro:include filename="$(find rl_subjugator_description)/urdf/xacro/collision.xacro"/>
+  <xacro:include filename="$(find rl_subjugator_description)/urdf/xacro/thruster.xacro"/>
+  <xacro:include filename="$(find rl_subjugator_description)/urdf/xacro/depth.xacro"/>
   <!-- Base Link of the Sub -->
   <link name="base_link">
@@ -25,5 +25,5 @@
       <origin rpy="0 0 0" xyz="0 0 0"/>
       <geometry>
-        <mesh filename="package://subjugator_description/urdf/meshes/Sub9.dae"/>
+        <mesh filename="package://rl_subjugator_description/urdf/meshes/Sub9.dae"/>
       </geometry>
     </visual>
@@ -31,5 +31,5 @@
     <collision name="buoyancy_collision">
       <!-- This collision is for calculating the buoyant forces-->
-      <origin rpy="0 0 0" xyz="0 0 0"/>
+      <origin rpy="0 0 0" xyz="0.354 0 0"/>
       <geometry>
         <sphere radius="0.1725"/>
@@ -97,4 +97,12 @@
   <!-- DVL Sensor -->
   <xacro:mil_dvl_sensor name="dvl_sensor" parent="base_link" xyz="0.3937 0 -0.2413" rpy="0 0 0"/>
+  <!-- Temp DVL Sensor to prevent crashing-->
+  <gazebo>
+    <plugin filename="gz-sim-odometry-publisher-system" name="gz::sim::systems::OdometryPublisher">
+      <odom_topic>/dvl/gt_odom</odom_topic>
+      <odom_frame_id>base_link</odom_frame_id>
+      <robot_base_frame_id>dvl_sensor_link</robot_base_frame_id>
+    </plugin>
+  </gazebo>
   <!-- IMU, Magnetometer -->
   <xacro:mil_imu_magnetometer
@@ -126,10 +134,3 @@
   <xacro:mil_thruster name="BRH" parent="base_link" xyz="0.127 -0.24765 0.053975" rpy="0 0 -0.523598776"/>
   <xacro:mil_thruster name="BLH" parent="base_link" xyz="0.127 0.24765 0.053975" rpy="0 0 0.523598776"/>
-  <!-- Damping -->
-  <gazebo reference="base_link">
-    <damping>
-      <linear>0.6</linear>
-      <angular>0.3</angular>
-    </damping>
-  </gazebo>
 </robot>

Commit message: Debloated rl_subjugator_description

File: src/subjugator/Reinforcement_Learning/src/rl_subjugator_description/urdf/sub9.urdf.xacro (robot description, xacro)
@@ -2,12 +2,11 @@
 <robot xmlns:xacro="http://www.ros.org/wiki/xacro" name="sub9">
   <!-- XACRO INCLUDES -->
-  <xacro:include filename="$(find rl_subjugator_description)/urdf/xacro/fixed_link.xacro"/>
-  <xacro:include filename="$(find rl_subjugator_description)/urdf/xacro/camera.xacro"/>
-  <xacro:include filename="$(find rl_subjugator_description)/urdf/xacro/imu_magnetometer.xacro"/>
-  <xacro:include filename="$(find rl_subjugator_description)/urdf/xacro/dvl.xacro"/>
-  <xacro:include filename="$(find rl_subjugator_description)/urdf/xacro/hydrophone.xacro"/>
-  <xacro:include filename="$(find rl_subjugator_description)/urdf/xacro/collision.xacro"/>
-  <xacro:include filename="$(find rl_subjugator_description)/urdf/xacro/thruster.xacro"/>
-  <xacro:include filename="$(find rl_subjugator_description)/urdf/xacro/depth.xacro"/>
+  <xacro:include filename="$(find subjugator_description)/urdf/xacro/fixed_link.xacro"/>
+  <xacro:include filename="$(find subjugator_description)/urdf/xacro/camera.xacro"/>
+  <xacro:include filename="$(find subjugator_description)/urdf/xacro/imu_magnetometer.xacro"/>
+  <xacro:include filename="$(find subjugator_description)/urdf/xacro/hydrophone.xacro"/>
+  <xacro:include filename="$(find subjugator_description)/urdf/xacro/collision.xacro"/>
+  <xacro:include filename="$(find subjugator_description)/urdf/xacro/thruster.xacro"/>
+  <xacro:include filename="$(find subjugator_description)/urdf/xacro/depth.xacro"/>
   <!-- Base Link of the Sub -->
   <link name="base_link">
@@ -25,5 +24,5 @@
       <origin rpy="0 0 0" xyz="0 0 0"/>
       <geometry>
-        <mesh filename="package://rl_subjugator_description/urdf/meshes/Sub9.dae"/>
+        <mesh filename="package://subjugator_description/urdf/meshes/Sub9.dae"/>
       </geometry>
     </visual>
@@ -95,6 +94,4 @@
   <xacro:mil_camera name="front_cam" parent="base_link" xyz="0.78 -0.014274 -0.050" rpy="0 0 0"/>
   <xacro:mil_camera name="down_cam" parent="base_link" xyz="0.45222 0.027913 -0.22" rpy="0 1.57 0"/>
-  <!-- DVL Sensor -->
-  <xacro:mil_dvl_sensor name="dvl_sensor" parent="base_link" xyz="0.3937 0 -0.2413" rpy="0 0 0"/>
   <!-- Temp DVL Sensor to prevent crashing-->
   <gazebo>
