Commit message: Added Underwater Camera Plugin

File: src/subjugator/simulation/subjugator_description/urdf/sub9.urdf.xacro (robot description, xacro)
@@ -1,11 +1,15 @@
 <?xml version="1.0" ?>
 <robot xmlns:xacro="http://www.ros.org/wiki/xacro" name="sub9">
-  <!-- Used for fixing robot to Gazebo 'base_link' -->
-  <link name="world"/>
+  <!-- XACRO INCLUDES -->
+  <xacro:include filename="$(find subjugator_description)/urdf/xacro/fixed_link.xacro"/>
+  <xacro:include filename="$(find subjugator_description)/urdf/xacro/camera.xacro"/>
+  <!-- KDL Parser does not like inertial base links, so use a 'fake' massless root link -->
+  <link name="base_link"/>
   <joint name="fixed" type="fixed">
-    <parent link="world"/>
-    <child link="base_link"/>
+    <parent link="base_link"/>
+    <child link="link1"/>
   </joint>
-  <link name="base_link">
+  <!-- Base Link of the Sub -->
+  <link name="link1">
     <inertial>
       <!-- Rough estimate of RoboSub 2022 -->
@@ -18,13 +22,19 @@
       <origin rpy="${pi/2} 0 ${pi}" xyz="${(0.915/2-0.009)} ${-(0.606/2)} ${-(0.381/2)}"/>
       <geometry>
-        <mesh filename="package://subjugator_description/urdf/meshes/sub9.dae"/>
+        <mesh filename="package://subjugator_description/urdf/meshes/sub9_redux.dae"/>
       </geometry>
     </visual>
     <collision name="collision">
-      <origin rpy="${pi/2} 0 ${pi}" xyz="${(0.915/2-0.009)} ${-(0.606/2)} ${-(0.381/2)}"/>
+    <!-- TODO: Need to add more accurate Collision Geometry -->
+    <origin rpy="0 0 0" xyz="-.05 0 0"/>
       <geometry>
-        <mesh filename="package://subjugator_description/urdf/meshes/sub9.dae"/>
+        <box size="0.8 0.3 0.36"/>
       </geometry>
     </collision>
   </link>
+  <!-- Sensors -->
+  <xacro:mil_fixed_link name="front_stereo" parent="base_link" xyz="0.2559 0 0.1707" rpy="0 0 0"/>
+  <xacro:mil_camera name="front_left_cam" parent="front_stereo" namespace="/camera/front/left" xyz="0 0.0445 0" rpy="0 0 0"/>
+  <!-- <xacro:mil_camera name="front_right_cam" parent="front_stereo" namespace="/camera/front/right" xyz="0 -0.0445 0" rpy="0 0 0"/>
+  <xacro:mil_camera name="down_left_cam" parent="base_link" namespace="/camera/down" xyz="0.054 0.105 -0.256" rpy="0 1.57 1.57"/> -->
 </robot>

File: src/subjugator/simulation/subjugator_description/urdf/xacro/camera.xacro (robot description, xacro)
@@ -1,29 +1,25 @@
 <?xml version="1.0"?>
 <robot xmlns:xacro="http://ros.org/wiki/xacro">
-  <!-- Macro for inserting an camera -->
+  <!-- Macro for inserting a camera -->
   <xacro:macro
     name="mil_camera"
-    params="name namespace:='/camera'
-                        parent='base_link' xyz:='0 0 0' rpy:='0 0 0'
-                        width:=960 height:=600 fov:=1.047 fps:=30
-                        k1:=0 k2:=0 t1:=0 t2:=0 k3:=0"
+    params="name namespace='/camera'
+                        parent='base_link' xyz='0 0 0' rpy='0 0 0'
+                        width=960 height=600 fov=1.047 fps=30
+                        k1=0 k2=0 t1=0 t2=0 k3=0"
   >
-    <link name="${name}"/>
-    <joint name="${name}_to_${parent}" type="fixed">
+    <link name="${name}_link"/>
+    <joint name="${name}_joint" type="fixed">
       <parent link="${parent}"/>
-      <child link="${name}"/>
+      <child link="${name}_link"/>
       <origin xyz="${xyz}" rpy="${rpy}"/>
     </joint>
-    <link name="${name}_optical"/>
-    <joint name="${name}_to_${name}_optical" type="fixed">
-      <parent link="${name}"/>
-      <child link="${name}_optical"/>
-      <origin xyz="0 0 0" rpy="${-pi/2} 0 ${-pi/2}"/>
-    </joint>
-    <gazebo reference="${name}">
-      <sensor name="${name}_sensor" type="camera">
+    <gazebo reference="${name}_link">
+      <sensor name="${name}_camera" type="rgbd_camera">
         <update_rate>${fps}</update_rate>
-        <camera name="${name}_camera">
-          <pose>0 0 0 0 0 0</pose>
+        <visualize>true</visualize>
+        <always_on>1</always_on>
+        <topic>${namespace}/image_raw</topic>
+        <camera>
           <horizontal_fov>${fov}</horizontal_fov>
           <image>
@@ -31,20 +27,19 @@
             <height>${height}</height>
           </image>
-          <distortion>
-            <k1>${k1}</k1>
-            <k2>${k2}</k2>
-            <k3>${k3}</k3>
-            <p1>${t1}</p1>
-            <p2>${t2}</p2>
-          </distortion>
+          <clip>
+            <near>0.1</near>
+            <far>10.0</far>
+          </clip>
         </camera>
-        <plugin name="${name}_controller" filename="libgazebo_ros_camera.so">
-          <ros>
-            <namespace>${namespace}</namespace>
-            <remapping>image_raw:=image_raw</remapping>
-            <remapping>camera_info:=camera_info</remapping>
-          </ros>
-          <cameraName>${namespace}</cameraName>
-          <frameName>${name}_optical</frameName>
+        <plugin
+          filename="UnderwaterCamera"
+          name="dave_gz_sensor_plugins::UnderwaterCamera">
+          <attenuationR>0.8</attenuationR>
+          <attenuationG>0.5</attenuationG>
+          <attenuationB>0.2</attenuationB>
+          <!-- Murky Coastal Waters -->
+          <backgroundR>85</backgroundR>
+          <backgroundG>107</backgroundG>
+          <backgroundB>47</backgroundB>
         </plugin>
       </sensor>

Commit message: added hydrodynamics plugin

File: src/subjugator/simulation/subjugator_description/urdf/sub9.urdf.xacro (robot description, xacro)
@@ -13,9 +13,6 @@
   <link name="link1">
     <inertial>
-      <!-- Rough estimate of RoboSub 2022 -->
       <mass value="21.5"/>
-      <!-- Estimate of inertial tensor based on inertial tensor for rectangular prism -->
-      <!-- https://en.wikipedia.org/wiki/List_of_moments_of_inertia#List_of_3D_inertia_tensors -->
-      <inertia ixx="0.96105" ixy="0.003" ixz="-0.02" iyy="1.799" iyz="0.0003" izz="2.1286"/>
+      <inertia ixx="0.96105" ixy="0" ixz="0" iyy="1.799" iyz="0" izz="2.1286"/>
     </inertial>
     <visual name="visual">
@@ -25,7 +22,7 @@
       </geometry>
     </visual>
+    <!-- TODO: Need to add more accurate Collision Geometry -->
     <collision name="collision">
-    <!-- TODO: Need to add more accurate Collision Geometry -->
-    <origin rpy="0 0 0" xyz="-.05 0 0"/>
+      <origin rpy="0 0 0" xyz="0 0 0"/>
       <geometry>
         <box size="0.8 0.3 0.36"/>
@@ -33,4 +30,29 @@
     </collision>
   </link>
+  <gazebo>
+    <plugin
+        filename="gz-sim-hydrodynamics-system"
+        name="gz::sim::systems::Hydrodynamics">
+      <link_name>base_link</link_name>
+      <xDotU>-0.04876161</xDotU>
+      <yDotV>-1.26324739</yDotV>
+      <zDotW>-1.26324739</zDotW>
+      <kDotP>0</kDotP>
+      <mDotQ>-0.3346</mDotQ>
+      <nDotR>-0.3346</nDotR>
+      <xUabsU>-0.62282</xUabsU>
+      <xU>-5</xU>
+      <yVabsV>-60.127</yVabsV>
+      <yV>-5</yV>
+      <zWabsW>-6.0127</zWabsW>
+      <zW>-100</zW>
+      <kPabsP>-0.001916</kPabsP>
+      <kP>-1</kP>
+      <mQabsQ>-6.32698957</mQabsQ>
+      <mQ>-1</mQ>
+      <nRabsR>-6.32698957</nRabsR>
+      <nR>-1</nR>
+    </plugin>
+  </gazebo>
   <!-- Sensors -->
   <xacro:mil_fixed_link name="front_stereo" parent="base_link" xyz="0.2559 0 0.1707" rpy="0 0 0"/>

Commit message: began work on other plugins

File: src/subjugator/simulation/subjugator_description/urdf/sub9.urdf.xacro (robot description, xacro)
@@ -4,4 +4,6 @@
   <xacro:include filename="$(find subjugator_description)/urdf/xacro/fixed_link.xacro"/>
   <xacro:include filename="$(find subjugator_description)/urdf/xacro/camera.xacro"/>
+  <xacro:include filename="$(find subjugator_description)/urdf/xacro/imu_magnetometer.xacro"/>
+  <xacro:include filename="$(find subjugator_description)/urdf/xacro/dvl.xacro"/>
   <!-- KDL Parser does not like inertial base links, so use a 'fake' massless root link -->
   <link name="base_link"/>
@@ -60,3 +62,18 @@
   <!-- <xacro:mil_camera name="front_right_cam" parent="front_stereo" namespace="/camera/front/right" xyz="0 -0.0445 0" rpy="0 0 0"/>
   <xacro:mil_camera name="down_left_cam" parent="base_link" namespace="/camera/down" xyz="0.054 0.105 -0.256" rpy="0 1.57 1.57"/> -->
+  <xacro:mil_imu_magnetometer
+    name="imu"
+    parent="base_link"
+    imu_topic='/imu/data_raw'
+    xyz="0.21236 0.00254 -0.10233"
+    rpy="0 -1.571 0"
+    rate="210"
+    ax="0.015707963"
+    ay="0.015707963"
+    az="0.015707963"
+    lx="0.08825985"
+    ly="0.08825985"
+    lz="0.08825985"
+  />
+  <xacro:mil_dvl name="dvl" parent="base_link" xyz="0.0908 0 -0.2459" rpy="0 0 0.785" gazebo_offset="0 0 -1" rate="6.5"/>
 </robot>

File: src/subjugator/simulation/subjugator_description/urdf/xacro/camera.xacro (robot description, xacro)
@@ -20,5 +20,5 @@
         <visualize>true</visualize>
         <always_on>1</always_on>
-        <topic>${namespace}/image_raw</topic>
+        <topic>${namespace}</topic>
         <camera>
           <horizontal_fov>${fov}</horizontal_fov>

File: src/subjugator/simulation/subjugator_description/urdf/xacro/dvl.xacro (robot description, xacro)
@@ -1,6 +1,6 @@
 <?xml version="1.0"?>
-<robot xmlns:xacro="http://ros.org/wiki/xacro">
+<robot xmlns:xacro="http://ros.org/wiki/xacro" xmlns:experimental="http://sdformat.org/schemas/experimental" xmlns:gz="http://gazebosim.org/schema">
   <!-- Macro for inserting a dvl -->
-  <xacro:macro name="mil_dvl" params="name:=dvl parent:='base_link' xyz:='0 0 0' rpy='0 0 0' gazebo_offset=:='0 0 0' rate:=1">
+  <xacro:macro name="mil_dvl" params="name='dvl' parent='base_link' xyz='0 0 0' rpy='0 0 0' gazebo_offset='0 0 0' rate='1'">
     <link name="${name}"/>
     <joint name="${name}_joint" type="fixed">
@@ -10,26 +10,58 @@
     </joint>
     <gazebo reference="${name}">
-      <sensor type="ray" name="${name}_sensor">
-        <always_on>true</always_on>
-        <update_rate>${rate}</update_rate>
-        <ray>
-          <scan>
-            <horizontal>
-              <samples>1</samples>
-              <resolution>3</resolution>
-              <min_angle>-0.3</min_angle>
-              <max_angle>0.3</max_angle>
-            </horizontal>
-          </scan>
-          <range>
-            <min>0.05</min>
-            <max>200</max>
-          </range>
-        </ray>
-        <plugin name="${name}_plugin" filename="libmil_dvl_gazebo.so">
-          <frame_id>${name}</frame_id>
-          <offset>${gazebo_offset}</offset>
-        </plugin>
-      </sensor>
+      <experimental:params>
+        <sensor
+            name="teledyne_pathfinder_dvl"
+            type="custom" gz:type="dvl">
+          <pose>0 0 0 0 0 0</pose>
+          <always_on>1</always_on>
+          <update_rate>${rate}</update_rate>
+          <topic>/model/${parent}/dvl/velocity</topic>
+          <gz:dvl>
+            <type>phased_array</type>
+            <arrangement degrees="true">
+              <beam id="1">
+                <aperture>2</aperture>
+                <rotation>45</rotation>
+                <tilt>30</tilt>
+              </beam>
+              <beam>
+                <aperture>2</aperture>
+                <rotation>135</rotation>
+                <tilt>30</tilt>
+              </beam>
+              <beam>
+                <aperture>2</aperture>
+                <rotation>-45</rotation>
+                <tilt>30</tilt>
+              </beam>
+              <beam>
+                <aperture>2</aperture>
+                <rotation>-135</rotation>
+                <tilt>30</tilt>
+              </beam>
+            </arrangement>
+            <tracking>
+              <bottom_mode>
+                <when>best</when>
+                <noise type="gaussian">
+                  <!-- +/- 0.4 cm/s precision at 10 m/s within 2 stddevs -->
+                  <stddev>0.002</stddev>
+                </noise>
+                <visualize>false</visualize>
+              </bottom_mode>
+            </tracking>
+            <!-- Roughly 1 m resolution at a 100m -->
+            <resolution>0.01</resolution>
+            <maximum_range>100.</maximum_range>
+            <minimum_range>0.1</minimum_range>
+            <!-- ENU to SFM -->
+            <reference_frame>0 0 0 0 0 -1.570796</reference_frame>
+          </gz:dvl>
+          <plugin
+            filename="gz-sim-dvl-system"
+            name="gz::sim::systems::DopplerVelocityLogSystem"/>
+        </sensor>
+      </experimental:params>
     </gazebo>
   </xacro:macro>

Commit message: Switch Sub9 to lowpoly and add collision models

File: src/subjugator/simulation/subjugator_description/urdf/sub9.urdf.xacro (robot description, xacro)
@@ -6,4 +6,5 @@
   <xacro:include filename="$(find subjugator_description)/urdf/xacro/imu_magnetometer.xacro"/>
   <xacro:include filename="$(find subjugator_description)/urdf/xacro/dvl.xacro"/>
+  <xacro:include filename="$(find subjugator_description)/urdf/xacro/collision.xacro"/>
   <!-- KDL Parser does not like inertial base links, so use a 'fake' massless root link -->
   <link name="base_link"/>
@@ -19,16 +20,11 @@
     </inertial>
     <visual name="visual">
-      <origin rpy="${pi/2} 0 ${pi}" xyz="${(0.915/2-0.009)} ${-(0.606/2)} ${-(0.381/2)}"/>
+      <origin rpy="0 0 0" xyz="-0.1 0.0125 0"/>
       <geometry>
-        <mesh filename="package://subjugator_description/urdf/meshes/sub9_redux.dae"/>
+        <mesh filename="package://subjugator_description/urdf/meshes/sub9.dae"/>
       </geometry>
     </visual>
-    <!-- TODO: Need to add more accurate Collision Geometry -->
-    <collision name="collision">
-      <origin rpy="0 0 0" xyz="0 0 0"/>
-      <geometry>
-        <box size="0.8 0.3 0.36"/>
-      </geometry>
-    </collision>
+    <!-- Imports subjugator's collisions from seperate XACRO -->
+    <xacro:collision />
   </link>
   <gazebo>

Commit message: Added basic thruster functionality for Gazebo

File: src/subjugator/simulation/subjugator_description/urdf/sub9.urdf.xacro (robot description, xacro)
@@ -9,11 +9,29 @@
   <xacro:include filename="$(find subjugator_description)/urdf/xacro/thruster.xacro"/>
   <!-- KDL Parser does not like inertial base links, so use a 'fake' massless root link -->
-  <link name="base_link"/>
+  <!-- <link name="base_link"/>
   <joint name="fixed" type="fixed">
     <parent link="base_link"/>
     <child link="link1"/>
-  </joint>
+  </joint> -->
+<joint name="thrustjoint" type="revolute">
+  <origin xyz="0 0 1" rpy="0 0 0"/>
+    <parent link="base_link"/>
+    <child link="thrusterer"/>
+    <!-- <gazebo> -->
+      <limit effort="1000" lower="0.0" upper="0.548" velocity="0.5"/>
+      <axis xyz="0 0 1"/>
+    <!-- </gazebo>  -->
+</joint>
+<link name="thrusterer">
+    <pose>1 0 0 0 0 0</pose>
+    <inertial>
+      <pose>0 0 0 0 0 0</pose>
+      <mass value="0.1"/>
+      <origin xyz="0 0 1" />
+      <inertia ixx="0.001" iyy="0.001" izz="0.001" ixy="0" ixz="0" iyz="0"/>
+    </inertial>
+</link>
   <!-- Base Link of the Sub -->
-  <link name="link1">
+  <link name="base_link">
     <inertial>
       <mass value="21.5"/>

Commit message: created even more low poly version of the sub

File: src/subjugator/simulation/subjugator_description/urdf/sub9.urdf.xacro (robot description, xacro)
@@ -9,12 +9,12 @@
   <xacro:include filename="$(find subjugator_description)/urdf/xacro/thruster.xacro"/>
   <!-- KDL Parser does not like inertial base links, so use a 'fake' massless root link -->
-  <!-- <link name="base_link"/>
+  <link name="base_link"/>
   <joint name="fixed" type="fixed">
     <parent link="base_link"/>
     <child link="link1"/>
-  </joint> -->
+  </joint>
 <joint name="thrustjoint" type="revolute">
   <origin xyz="0 0 1" rpy="0 0 0"/>
-    <parent link="base_link"/>
+    <parent link="link1"/>
     <child link="thrusterer"/>
     <!-- <gazebo> -->
@@ -33,5 +33,5 @@
 </link>
   <!-- Base Link of the Sub -->
-  <link name="base_link">
+  <link name="link1">
     <inertial>
       <mass value="21.5"/>
@@ -39,11 +39,16 @@
     </inertial>
     <visual name="visual">
-      <origin rpy="0 0 0" xyz="-0.1 0.0125 0"/>
+      <origin rpy="0 0 0" xyz="-0.1 0.0125 -1"/>
       <geometry>
-        <mesh filename="package://subjugator_description/urdf/meshes/sub9.dae"/>
+        <mesh filename="package://subjugator_description/urdf/meshes/Sub9.dae"/>
       </geometry>
     </visual>
     <!-- Imports subjugator's collisions from seperate XACRO -->
-    <xacro:collision />
+    <collision name="main_collision">
+      <origin rpy="0 0 0" xyz="0 0 0"/>
+      <geometry>
+        <box size="0.945 0.35 0.4"/>
+      </geometry>
+    </collision>
   </link>
   <gazebo>
@@ -51,5 +56,5 @@
         filename="gz-sim-hydrodynamics-system"
         name="gz::sim::systems::Hydrodynamics">
-      <link_name>base_link</link_name>
+      <link_name>link1</link_name>
       <xDotU>-0.04876161</xDotU>
       <yDotV>-1.26324739</yDotV>
@@ -83,6 +88,6 @@
   </gazebo>
   <!-- Sensors -->
-  <xacro:mil_fixed_link name="front_stereo" parent="base_link" xyz="0.2559 0 0.1707" rpy="0 0 0"/>
-  <xacro:mil_camera name="front_left_cam" parent="front_stereo" namespace="/camera/front/left" xyz="-0.65 0 -0.3" rpy="0 0 9.5"/>
+  <xacro:mil_fixed_link name="front_stereo" parent="link1" xyz="0.2559 0 0.1707" rpy="0 0 0"/>
+  <!-- <xacro:mil_camera name="front_left_cam" parent="front_stereo" namespace="/camera/front/left" xyz="-0.65 0 -0.3" rpy="0 0 9.5"/> -->
   <!-- <xacro:mil_camera name="front_right_cam" parent="front_stereo" namespace="/camera/front/right" xyz="0 -0.0445 0" rpy="0 0 0"/>
   <xacro:mil_camera name="down_left_cam" parent="base_link" namespace="/camera/down" xyz="0.054 0.105 -0.256" rpy="0 1.57 1.57"/> -->
@@ -90,5 +95,5 @@
   <xacro:mil_dvl_sensor
     name="dvl_sensor"
-    parent="base_link"
+    parent="link1"
     xyz="0.21236 0.00254 -0.10233"
     rpy="0 0 0"
@@ -96,5 +101,5 @@
   <xacro:mil_imu_magnetometer
     name="imu"
-    parent="base_link"
+    parent="link1"
     imu_topic='/imu/data_raw'
     xyz="0.21236 0.00254 -0.10233"

File: src/subjugator/simulation/subjugator_description/urdf/xacro/new_dvl.xacro (robot description, xacro)
@@ -59,5 +59,5 @@
                 <stddev>0.015</stddev>
               </noise>
-              <visualize>false</visualize>
+              <visualize>true</visualize>
             </water_mass_mode>
             <bottom_mode>
@@ -66,5 +66,5 @@
                 <stddev>0.005</stddev>
               </noise>
-              <visualize>false</visualize>
+              <visualize>true</visualize>
             </bottom_mode>
           </tracking>
