Commit message: Placed all plugins and added ROS GZ bridges

File: src/subjugator/simulation/subjugator_description/urdf/sub9.urdf.xacro (robot description, xacro)
@@ -5,50 +5,34 @@
   <xacro:include filename="$(find subjugator_description)/urdf/xacro/camera.xacro"/>
   <xacro:include filename="$(find subjugator_description)/urdf/xacro/imu_magnetometer.xacro"/>
-  <xacro:include filename="$(find subjugator_description)/urdf/xacro/new_dvl.xacro"/>
+  <xacro:include filename="$(find subjugator_description)/urdf/xacro/dvl.xacro"/>
   <xacro:include filename="$(find subjugator_description)/urdf/xacro/collision.xacro"/>
   <xacro:include filename="$(find subjugator_description)/urdf/xacro/thruster.xacro"/>
-  <!-- KDL Parser does not like inertial base links, so use a 'fake' massless root link -->
-  <link name="base_link"/>
-  <joint name="fixed" type="fixed">
-    <parent link="base_link"/>
-    <child link="link1"/>
-  </joint>
-<joint name="thrustjoint" type="revolute">
-  <origin xyz="0 0 1" rpy="0 0 0"/>
-    <parent link="link1"/>
-    <child link="thrusterer"/>
-    <!-- <gazebo> -->
-      <limit effort="1000" lower="0.0" upper="0.548" velocity="0.5"/>
-      <axis xyz="0 0 1"/>
-    <!-- </gazebo>  -->
-</joint>
-<link name="thrusterer">
-    <pose>1 0 0 0 0 0</pose>
+  <!-- Base Link of the Sub -->
+  <link name="base_link">
+    <!-- Sub's Pose -->
+    <origin rpy="0 0 0" xyz="-0.1 0.0125 -1"/>
+    <!-- Inertial Properties -->
     <inertial>
-      <pose>0 0 0 0 0 0</pose>
-      <mass value="0.1"/>
-      <origin xyz="0 0 1" />
-      <inertia ixx="0.001" iyy="0.001" izz="0.001" ixy="0" ixz="0" iyz="0"/>
+      <origin rpy="0 0 0" xyz="0 0 0"/>
+      <!-- Need to be properly caluclated at some point -->
+      <mass value="30.5"/>
+      <inertia ixx="0.96105" ixy="0.003" ixz="-0.02" iyy="1.799" iyz="0.0003" izz="2.1286"/>
     </inertial>
-</link>
-  <!-- Base Link of the Sub -->
-  <link name="link1">
-    <inertial>
-      <mass value="21.5"/>
-      <inertia ixx="0.96105" ixy="0" ixz="0" iyy="1.799" iyz="0" izz="2.1286"/>
-    </inertial>
+    <!-- Visual Data-->
     <visual name="visual">
-      <origin rpy="0 0 0" xyz="-0.1 0.0125 -1"/>
+      <origin rpy="0 0 0" xyz="0 0 0"/>
       <geometry>
         <mesh filename="package://subjugator_description/urdf/meshes/Sub9.dae"/>
       </geometry>
     </visual>
-    <!-- Imports subjugator's collisions from seperate XACRO -->
+    <!-- Collision Data -->
     <collision name="main_collision">
-      <origin rpy="0 0 0" xyz="0 0 0"/>
+      <!-- This collision is for calculating the buoyant forces-->
+      <origin rpy="0 0 0" xyz="0 0 0.1"/>
       <geometry>
-        <box size="0.945 0.35 0.4"/>
+        <box size="0.9 0.35 0.2"/>
       </geometry>
     </collision>
+    <!-- Need to add 'shell' collisions-->
   </link>
   <gazebo>
@@ -56,52 +40,41 @@
         filename="gz-sim-hydrodynamics-system"
         name="gz::sim::systems::Hydrodynamics">
-      <link_name>link1</link_name>
-      <xDotU>-0.04876161</xDotU>
-      <yDotV>-1.26324739</yDotV>
-      <zDotW>-1.26324739</zDotW>
-      <kDotP>0</kDotP>
-      <mDotQ>-0.3346</mDotQ>
-      <nDotR>-0.3346</nDotR>
-      <xUabsU>-0.62282</xUabsU>
-      <xU>-5</xU>
-      <yVabsV>-60.127</yVabsV>
-      <yV>-5</yV>
-      <zWabsW>-6.0127</zWabsW>
-      <zW>-100</zW>
-      <kPabsP>-0.001916</kPabsP>
-      <kP>-1</kP>
-      <mQabsQ>-6.32698957</mQabsQ>
-      <mQ>-1</mQ>
-      <nRabsR>-6.32698957</nRabsR>
-      <nR>-1</nR>
-    </plugin>
-    <plugin
-      filename="gz-sim-thruster-system"
-      name="gz::sim::systems::Thruster">
-      <namespace>thrustme</namespace>
-      <use_angvel_cmd>0</use_angvel_cmd>
-      <joint_name>thrustjoint</joint_name>
-      <thrust_coefficient>0.004422</thrust_coefficient>
-      <fluid_density>1000</fluid_density>
-      <propeller_diameter>0.2</propeller_diameter>
+      <link_name>base_link</link_name>
+      <xDotU>-2</xDotU>
+      <yDotV>-5</yDotV>
+      <zDotW>-5</zDotW>
+      <kDotP>-0.1</kDotP>
+      <mDotQ>-1</mDotQ>
+      <nDotR>-1</nDotR>
+      <xUabsU>-25</xUabsU>
+      <xU>-50</xU>
+      <yVabsV>-25</yVabsV>
+      <yV>-50</yV>
+      <zWabsW>-5</zWabsW>
+      <zW>-50</zW>
+      <kPabsP>-5</kPabsP>
+      <kP>-10</kP>
+      <mQabsQ>-5</mQabsQ>
+      <mQ>-10</mQ>
+      <nRabsR>-5</nRabsR>
+      <nR>-10</nR>
     </plugin>
   </gazebo>
-  <!-- Sensors -->
-  <xacro:mil_fixed_link name="front_stereo" parent="link1" xyz="0.2559 0 0.1707" rpy="0 0 0"/>
-  <!-- <xacro:mil_camera name="front_left_cam" parent="front_stereo" namespace="/camera/front/left" xyz="-0.65 0 -0.3" rpy="0 0 9.5"/> -->
-  <!-- <xacro:mil_camera name="front_right_cam" parent="front_stereo" namespace="/camera/front/right" xyz="0 -0.0445 0" rpy="0 0 0"/>
-  <xacro:mil_camera name="down_left_cam" parent="base_link" namespace="/camera/down" xyz="0.054 0.105 -0.256" rpy="0 1.57 1.57"/> -->
-  <!-- DVL Sensor-->
+  <!-- Cameras -->
+  <xacro:mil_camera name="front_cam" parent="base_link" xyz="-0.25 -0.014274 -0.018" rpy="0 0 3.14159"/>
+  <xacro:mil_camera name="down_cam" parent="base_link" xyz="-0.15222 0.027913 -0.16" rpy="0 1.57 0"/>
+  <!-- DVL Sensor -->
   <xacro:mil_dvl_sensor
     name="dvl_sensor"
-    parent="link1"
+    parent="base_link"
     xyz="0.21236 0.00254 -0.10233"
     rpy="0 0 0"
   />
+   <!-- IMU, Magnetometer -->
   <xacro:mil_imu_magnetometer
     name="imu"
-    parent="link1"
-    imu_topic='/imu/data_raw'
-    xyz="0.21236 0.00254 -0.10233"
+    namespace='/imu'
+    parent="base_link"
+    xyz="0.0632 -0.164 -0.079"
     rpy="0 -1.571 0"
     rate="210"
@@ -113,3 +86,61 @@
     lz="0.08825985"
   />
+   <!-- Thrusters -->
+   <!-- Need to test these orientations!-->
+  <xacro:mil_thruster
+    name="FLH"
+    parent="base_link"
+    xyz="-0.15217 -0.16474 0.010449"
+    rpy="0 0 0"
+    dir_rpy="0 0 0"
+  />
+  <xacro:mil_thruster
+    name="FRH"
+    parent="base_link"
+    xyz="-0.1492 0.13821 0.010449"
+    rpy="0 0 0"
+    dir_rpy="0 0 0"
+  />
+  <xacro:mil_thruster
+    name="BRH"
+    parent="base_link"
+    xyz="0.31117 0.13821 0.010449"
+    rpy="0 0 0"
+    dir_rpy="0 0 0"
+  />
+  <xacro:mil_thruster
+    name="BLH"
+    parent="base_link"
+    xyz="0.30868 -0.16621 0.010449"
+    rpy="0 0 0"
+    dir_rpy="0 0 0"
+  />
+  <xacro:mil_thruster
+    name="FLV"
+    parent="base_link"
+    xyz="-0.14714 -0.26409 0.038317"
+    rpy="-1.5708 0 0"
+    dir_rpy="0 0 0"
+  />
+  <xacro:mil_thruster
+    name="FRV"
+    parent="base_link"
+    xyz="-0.147 0.2413 0.038324"
+    rpy="1.5708 0 0"
+    dir_rpy="0 0 0"
+  />
+  <xacro:mil_thruster
+    name="BRV"
+    parent="base_link"
+    xyz="0.32369 0.22645 0.038317"
+    rpy="1.5708 0 0"
+    dir_rpy="0 0 0"
+  />
+  <xacro:mil_thruster
+    name="BLV"
+    parent="base_link"
+    xyz="0.32397 -0.25204 0.038324"
+    rpy="-1.5708 0 0"
+    dir_rpy="0 0 0"
+  />
 </robot>

File: src/subjugator/simulation/subjugator_description/urdf/xacro/camera.xacro (robot description, xacro)
@@ -4,15 +4,28 @@
   <xacro:macro
     name="mil_camera"
-    params="name namespace='/camera'
-                        parent='base_link' xyz='0 0 0' rpy='0 0 0'
-                        width=960 height=600 fov=1.047 fps=30
-                        k1=0 k2=0 t1=0 t2=0 k3=0"
+    params="name parent xyz rpy
+            use_image_processing=false
+            width=960 height=600 fov=1.047 fps=30"
   >
-    <link name="${name}_link"/>
+    <!-- Camera Link -->
+     <link name="${name}_link">
+      <origin xyz="0 0 0" rpy="0 0 0"/>
+      <inertial>
+        <origin xyz="0 0 0" rpy="0 0 0"/>
+        <mass value="0.1"/>
+        <inertia ixx="0.001" iyy="0.001" izz="0.001" ixy="0" ixz="0" iyz="0"/>
+      </inertial>
+    </link>
+    <!-- Camera Joint -->
     <joint name="${name}_joint" type="fixed">
+      <origin xyz="${xyz}" rpy="${rpy}"/>
       <parent link="${parent}"/>
       <child link="${name}_link"/>
-      <origin xyz="${xyz}" rpy="${rpy}"/>
     </joint>
+    <!-- This ensures that the fixed link is not simplified away -->
+    <gazebo reference="${name}_joint">
+      <disableFixedJointLumping>true</disableFixedJointLumping>
+      <preserveFixedJoint>true</preserveFixedJoint>
+    </gazebo>
     <gazebo reference="${name}_link">
       <sensor name="${name}_camera" type="rgbd_camera">
@@ -20,5 +33,5 @@
         <visualize>true</visualize>
         <always_on>1</always_on>
-        <topic>${namespace}</topic>
+        <topic>${name}</topic>
         <camera>
           <horizontal_fov>${fov}</horizontal_fov>
@@ -32,15 +45,17 @@
           </clip>
         </camera>
-        <plugin
-          filename="UnderwaterCamera"
-          name="dave_gz_sensor_plugins::UnderwaterCamera">
-          <attenuationR>0.8</attenuationR>
-          <attenuationG>0.5</attenuationG>
-          <attenuationB>0.2</attenuationB>
-          <!-- Murky Coastal Waters -->
-          <backgroundR>85</backgroundR>
-          <backgroundG>107</backgroundG>
-          <backgroundB>47</backgroundB>
-        </plugin>
+        <xacro:if value="${use_image_processing}">
+          <plugin
+            filename="UnderwaterCamera"
+            name="dave_gz_sensor_plugins::UnderwaterCamera">
+            <attenuationR>0.8</attenuationR>
+            <attenuationG>0.5</attenuationG>
+            <attenuationB>0.2</attenuationB>
+            <!-- Murky Coastal Waters -->
+            <backgroundR>85</backgroundR>
+            <backgroundG>107</backgroundG>
+            <backgroundB>47</backgroundB>
+          </plugin>
+        </xacro:if>
       </sensor>
     </gazebo>

File: src/subjugator/simulation/subjugator_description/urdf/xacro/dvl.xacro (robot description, xacro)
@@ -1,68 +1,95 @@
 <?xml version="1.0"?>
 <robot xmlns:xacro="http://ros.org/wiki/xacro" xmlns:experimental="http://sdformat.org/schemas/experimental" xmlns:gz="http://gazebosim.org/schema">
-  <!-- Macro for inserting a dvl -->
-  <xacro:macro name="mil_dvl" params="name='dvl' parent='base_link' xyz='0 0 0' rpy='0 0 0' gazebo_offset='0 0 0' rate='1'">
-    <link name="${name}"/>
+  <!-- Macro for inserting a DVL -->
+  <xacro:macro
+    name="mil_dvl_sensor"
+    params="name parent xyz rpy"
+  >
+    <!-- DVL Link -->
+     <link name="${name}_link">
+      <origin xyz="0 0 0" rpy="0 0 0"/>
+      <inertial>
+        <origin xyz="0 0 0" rpy="0 0 0"/>
+        <mass value="0.1"/>
+        <inertia ixx="0.001" iyy="0.001" izz="0.001" ixy="0" ixz="0" iyz="0"/>
+      </inertial>
+    </link>
+    <!-- DVL Joint -->
     <joint name="${name}_joint" type="fixed">
       <origin xyz="${xyz}" rpy="${rpy}"/>
       <parent link="${parent}"/>
-      <child link="${name}"/>
+      <child link="${name}_link"/>
     </joint>
-    <gazebo reference="${name}">
-      <experimental:params>
-        <sensor
-            name="teledyne_pathfinder_dvl"
-            type="custom" gz:type="dvl">
-          <pose>0 0 0 0 0 0</pose>
-          <always_on>1</always_on>
-          <update_rate>${rate}</update_rate>
-          <topic>/model/${parent}/dvl/velocity</topic>
-          <gz:dvl>
-            <type>phased_array</type>
-            <arrangement degrees="true">
-              <beam id="1">
-                <aperture>2</aperture>
-                <rotation>45</rotation>
-                <tilt>30</tilt>
-              </beam>
-              <beam>
-                <aperture>2</aperture>
-                <rotation>135</rotation>
-                <tilt>30</tilt>
-              </beam>
-              <beam>
-                <aperture>2</aperture>
-                <rotation>-45</rotation>
-                <tilt>30</tilt>
-              </beam>
-              <beam>
-                <aperture>2</aperture>
-                <rotation>-135</rotation>
-                <tilt>30</tilt>
-              </beam>
-            </arrangement>
-            <tracking>
-              <bottom_mode>
-                <when>best</when>
-                <noise type="gaussian">
-                  <!-- +/- 0.4 cm/s precision at 10 m/s within 2 stddevs -->
-                  <stddev>0.002</stddev>
-                </noise>
-                <visualize>false</visualize>
-              </bottom_mode>
-            </tracking>
-            <!-- Roughly 1 m resolution at a 100m -->
-            <resolution>0.01</resolution>
-            <maximum_range>100.</maximum_range>
-            <minimum_range>0.1</minimum_range>
-            <!-- ENU to SFM -->
-            <reference_frame>0 0 0 0 0 -1.570796</reference_frame>
-          </gz:dvl>
-          <plugin
-            filename="gz-sim-dvl-system"
-            name="gz::sim::systems::DopplerVelocityLogSystem"/>
-        </sensor>
-      </experimental:params>
+    <!-- This ensures that the fixed link is not simplified away -->
+    <gazebo reference="${name}_joint">
+      <disableFixedJointLumping>true</disableFixedJointLumping>
+      <preserveFixedJoint>true</preserveFixedJoint>
     </gazebo>
-  </xacro:macro>
+    <!-- Sensor/Plugin Info-->
+    <gazebo reference="${name}_link">
+      <sensor
+        name="A50_Waterlinked" type="custom"
+        gz:type="dvl">
+        <pose>0 0 0 0 0 0</pose>
+        <always_on>1</always_on>
+        <update_rate>8</update_rate>
+        <topic>/dvl/velocity</topic>
+        <gz:dvl>
+          <type>phased_array</type>
+          <arrangement degrees="true">
+            <beam id="1">
+              <aperture>3</aperture>
+              <rotation>-135</rotation>
+              <tilt>25</tilt>
+            </beam>
+            <beam>
+              <aperture>3</aperture>
+              <rotation>135</rotation>
+              <tilt>25</tilt>
+            </beam>
+            <beam>
+              <aperture>3</aperture>
+              <rotation>45</rotation>
+              <tilt>25</tilt>
+            </beam>
+            <beam>
+              <aperture>3</aperture>
+              <rotation>-45</rotation>
+              <tilt>25</tilt>
+            </beam>
+          </arrangement>
+          <tracking>
+            <water_mass_mode>
+              <when>best</when>
+              <water_velocity>
+                <x>0.</x>
+                <y>0.</y>
+                <z>0.</z>
+              </water_velocity>
+              <boundaries>
+                <near>10.</near>
+                <far>100.</far>
+              </boundaries>
+              <bins>10</bins>
+              <noise type="gaussian">
+                <stddev>0.015</stddev>
+              </noise>
+              <visualize>true</visualize>
+            </water_mass_mode>
+            <bottom_mode>
+              <when>best</when>
+              <noise type="gaussian">
+                <stddev>0.005</stddev>
+              </noise>
+              <visualize>true</visualize>
+            </bottom_mode>
+          </tracking>
+          <maximum_range>200.</maximum_range>
+          <minimum_range>0.3</minimum_range>
+          <!-- ENU to FSD -->
+          <reference_frame>0 0 0 3.14 0 -1.57</reference_frame>
+        </gz:dvl>
+      </sensor>
+    </gazebo>
+    </xacro:macro>
 </robot>

File: src/subjugator/simulation/subjugator_description/urdf/xacro/imu_magnetometer.xacro (robot description, xacro)
@@ -3,17 +3,33 @@
   <xacro:macro
     name="mil_imu_magnetometer"
-    params="name parent imu_topic xyz rpy rate ax ay az lx ly lz"
+    params="name namespace parent xyz rpy
+            rate ax ay az lx ly lz"
   >
-    <link name="${name}"/>
+   <!-- Imu link -->
+   <link name="${name}_link">
+      <origin xyz="0 0 0" rpy="0 0 0"/>
+      <inertial>
+        <origin xyz="0 0 0" rpy="0 0 0"/>
+        <mass value="0.1"/>
+        <inertia ixx="0.001" iyy="0.001" izz="0.001" ixy="0" ixz="0" iyz="0"/>
+      </inertial>
+    </link>
+    <!-- IMU joint -->
     <joint name="${name}_joint" type="fixed">
       <origin xyz="${xyz}" rpy="${rpy}"/>
       <parent link="${parent}"/>
-      <child link="${name}"/>
+      <child link="${name}_link"/>
     </joint>
-    <gazebo reference="${name}">
-      <sensor name="${name}_imu_sensor" type="imu">
+    <!-- This ensures that the fixed link is not simplified away -->
+    <gazebo reference="${name}_joint">
+      <disableFixedJointLumping>true</disableFixedJointLumping>
+      <preserveFixedJoint>true</preserveFixedJoint>
+    </gazebo>
+    <!-- Sensor/Plugin Info-->
+    <gazebo reference="${name}_link">
+      <sensor name="VectorNav_IMU" type="imu">
         <always_on>true</always_on>
         <update_rate>${rate}</update_rate>
-        <topic>${imu_topic}/imu</topic>
+        <topic>${namespace}/data_raw</topic>
         <imu>
           <linear_acceleration>
@@ -57,8 +73,8 @@
         </plugin>
       </sensor>
-      <sensor name="${name}_mag_sensor" type="magnetometer">
+      <sensor name="VectorNav_MAG" type="magnetometer">
         <always_on>true</always_on>
         <update_rate>${rate}</update_rate>
-        <topic>${imu_topic}/imu_mag</topic>
+        <topic>${namespace}/mag</topic>
         <plugin
             filename="gz-sim-magnetometer-system"

File: src/subjugator/simulation/subjugator_description/urdf/xacro/thruster.xacro (robot description, xacro)
@@ -1,29 +1,60 @@
 <?xml version="1.0"?>
 <robot xmlns:xacro="http://www.ros.org/wiki/xacro">
-  <xacro:macro name="mil_thruster" params="name parent xyz rpy">
-    <!-- Define the thruster link -->
-    <link name="${name}_link">
+  <!-- Macro for inserting a Thruster -->
+  <xacro:macro
+    name="mil_thruster"
+    params="name parent xyz rpy
+            dir_rpy">
+    <!-- Link for base of thruster (this is for TF) -->
+     <link name="${name}_link">
+      <origin xyz="0 0 0" rpy="0 0 0"/>
       <inertial>
-        <mass value="0.1"/>  <!-- Add some mass to avoid physics issues -->
-        <origin xyz="0 0 0" />
+        <origin xyz="0 0 0" rpy="0 0 0"/>
+        <mass value="0.1"/>
         <inertia ixx="0.001" iyy="0.001" izz="0.001" ixy="0" ixz="0" iyz="0"/>
       </inertial>
     </link>
-    <!-- Define the joint -->
+    <!-- Thruster base Joint -->
     <joint name="${name}_joint" type="fixed">
+      <origin xyz="${xyz}" rpy="${rpy}"/>
       <parent link="${parent}"/>
       <child link="${name}_link"/>
-      <origin xyz="${xyz}" rpy="${rpy}"/>
     </joint>
-    <!-- Define Gazebo plugin -->
+    <!-- This ensures that the fixed link is not simplified away -->
+    <gazebo reference="${name}_joint">
+      <disableFixedJointLumping>true</disableFixedJointLumping>
+      <preserveFixedJoint>true</preserveFixedJoint>
+    </gazebo>
+    <!-- Thruster Direction link (this is for the plugin) -->
+    <!-- The plugin does not work with a fixed link -->
+    <link name="${name}_dir_link">
+      <origin xyz="0 0 0" rpy="0 0 0"/>
+      <inertial>
+        <origin xyz="0 0 0" rpy="0 0 0"/>
+        <mass value="0.1"/>
+        <inertia ixx="0.001" iyy="0.001" izz="0.001" ixy="0" ixz="0" iyz="0"/>
+      </inertial>
+    </link>
+    <!-- Thruster Direction joint -->
+    <joint name="${name}_dir_joint" type="revolute">
+      <origin xyz="0 0 1" rpy="${dir_rpy}"/>
+      <parent link="${name}_link"/>
+      <child link="${name}_dir_link"/>
+      <limit effort="1000" lower="0.0" upper="0.548" velocity="0.5"/>
+      <axis xyz="0 0 1"/>
+    </joint>
+    <!-- Sensor/Plugin Info-->
+    <!-- For the thruster plugin this gazebo tag needs to be global-->
+    <!-- Don't give it a reference like the other plugins-->
     <gazebo>
-      <plugin filename="gz-sim-thruster-system" name="gz::sim::systems::Thruster">
+      <plugin
+        filename="gz-sim-thruster-system"
+        name="gz::sim::systems::Thruster">
         <namespace>${name}</namespace>
         <use_angvel_cmd>0</use_angvel_cmd>
-        <joint_name>${name}_joint</joint_name>
-        <thrust_coefficient>0.004422</thrust_coefficient>
+        <joint_name>${name}_dir_joint</joint_name>
+        <thrust_coefficient>0.01407</thrust_coefficient>
         <fluid_density>1000</fluid_density>
         <propeller_diameter>0.2</propeller_diameter>
-        <debug>true</debug>
       </plugin>
     </gazebo>

Commit message: Verified Axis directions and orientation

File: src/subjugator/simulation/subjugator_description/urdf/sub9.urdf.xacro (robot description, xacro)
@@ -94,5 +94,4 @@
     xyz="-0.15217 -0.16474 0.010449"
     rpy="0 0 0"
-    dir_rpy="0 0 0"
   />
   <xacro:mil_thruster
@@ -101,5 +100,4 @@
     xyz="-0.1492 0.13821 0.010449"
     rpy="0 0 0"
-    dir_rpy="0 0 0"
   />
   <xacro:mil_thruster
@@ -108,5 +106,4 @@
     xyz="0.31117 0.13821 0.010449"
     rpy="0 0 0"
-    dir_rpy="0 0 0"
   />
   <xacro:mil_thruster
@@ -115,5 +112,4 @@
     xyz="0.30868 -0.16621 0.010449"
     rpy="0 0 0"
-    dir_rpy="0 0 0"
   />
   <xacro:mil_thruster
@@ -121,6 +117,5 @@
     parent="base_link"
     xyz="-0.14714 -0.26409 0.038317"
-    rpy="-1.5708 0 0"
-    dir_rpy="0 0 0"
+    rpy="-1.5708 0 0.7854"
   />
   <xacro:mil_thruster
@@ -128,6 +123,5 @@
     parent="base_link"
     xyz="-0.147 0.2413 0.038324"
-    rpy="1.5708 0 0"
-    dir_rpy="0 0 0"
+    rpy="1.5708 0 -0.7854"
   />
   <xacro:mil_thruster
@@ -135,6 +129,5 @@
     parent="base_link"
     xyz="0.32369 0.22645 0.038317"
-    rpy="1.5708 0 0"
-    dir_rpy="0 0 0"
+    rpy="-1.5708 0 0.7854"
   />
   <xacro:mil_thruster
@@ -142,6 +135,5 @@
     parent="base_link"
     xyz="0.32397 -0.25204 0.038324"
-    rpy="-1.5708 0 0"
-    dir_rpy="0 0 0"
+    rpy="1.5708 0 -0.7854"
   />
 </robot>

File: src/subjugator/simulation/subjugator_description/urdf/xacro/thruster.xacro (robot description, xacro)
@@ -4,6 +4,5 @@
   <xacro:macro
     name="mil_thruster"
-    params="name parent xyz rpy
-            dir_rpy">
+    params="name parent xyz rpy">
     <!-- Link for base of thruster (this is for TF) -->
      <link name="${name}_link">
@@ -11,5 +10,5 @@
       <inertial>
         <origin xyz="0 0 0" rpy="0 0 0"/>
-        <mass value="0.1"/>
+        <mass value="0.01"/>
         <inertia ixx="0.001" iyy="0.001" izz="0.001" ixy="0" ixz="0" iyz="0"/>
       </inertial>
@@ -32,5 +31,5 @@
       <inertial>
         <origin xyz="0 0 0" rpy="0 0 0"/>
-        <mass value="0.1"/>
+        <mass value="0.01"/>
         <inertia ixx="0.001" iyy="0.001" izz="0.001" ixy="0" ixz="0" iyz="0"/>
       </inertial>
@@ -38,5 +37,5 @@
     <!-- Thruster Direction joint -->
     <joint name="${name}_dir_joint" type="revolute">
-      <origin xyz="0 0 1" rpy="${dir_rpy}"/>
+      <origin xyz="0 0 1" rpy="0 0 0"/>
       <parent link="${name}_link"/>
       <child link="${name}_dir_link"/>
