Commit message: subjugator_localization: added packaged for ukf filtering and odometry; updated DVL and IMU gazebo sensors

File: src/subjugator/simulation/subjugator_description/urdf/sub9.urdf.xacro (robot description, xacro)
@@ -1,3 +1,3 @@
-<?xml version="1.0" ?>
+<?xml version="1.0"?>
 <robot xmlns:xacro="http://www.ros.org/wiki/xacro" name="sub9">
   <!-- XACRO INCLUDES -->
@@ -15,5 +15,5 @@
     <inertial>
       <origin rpy="0 0 0" xyz="0 0 0"/>
-      <!-- Need to be properly caluclated at some point -->
+      <!-- Need to be properly calculated at some point -->
       <mass value="30.5"/>
       <inertia ixx="0.96105" ixy="0.003" ixz="-0.02" iyy="1.799" iyz="0.0003" izz="2.1286"/>
@@ -37,7 +37,5 @@
   </link>
   <gazebo>
-    <plugin
-        filename="gz-sim-hydrodynamics-system"
-        name="gz::sim::systems::Hydrodynamics">
+    <plugin filename="gz-sim-hydrodynamics-system" name="gz::sim::systems::Hydrodynamics">
       <link_name>base_link</link_name>
       <xDotU>-2</xDotU>
@@ -62,24 +60,9 @@
   </gazebo>
   <!-- Cameras -->
-  <xacro:mil_camera
-    name="front_cam"
-    parent="base_link"
-    xyz="-0.32 -0.014274 -0.050"
-    rpy="0 0 3.14159"
-  />
-  <xacro:mil_camera
-    name="down_cam"
-    parent="base_link"
-    xyz="-0.15222 0.027913 -0.22"
-    rpy="0 1.57 0"
-  />
+  <xacro:mil_camera name="front_cam" parent="base_link" xyz="-0.32 -0.014274 -0.050" rpy="0 0 3.14159"/>
+  <xacro:mil_camera name="down_cam" parent="base_link" xyz="-0.15222 0.027913 -0.22" rpy="0 1.57 0"/>
   <!-- DVL Sensor -->
-  <xacro:mil_dvl_sensor
-    name="dvl_sensor"
-    parent="base_link"
-    xyz="0.21236 0.00254 -0.10233"
-    rpy="0 0 0"
-  />
-   <!-- IMU, Magnetometer -->
+  <xacro:mil_dvl_sensor name="dvl_sensor" parent="base_link" xyz="0.21236 0.00254 -0.10233" rpy="0 0 0"/>
+  <!-- IMU, Magnetometer -->
   <xacro:mil_imu_magnetometer
     name="imu"
@@ -87,5 +70,5 @@
     parent="base_link"
     xyz="0.0632 -0.164 -0.079"
-    rpy="0 -1.571 0"
+    rpy="0 0 0"
     rate="210"
     ax="0.015707963"
@@ -96,54 +79,14 @@
     lz="0.08825985"
   />
-   <!-- Thrusters -->
-   <!-- Front/Back Left/Right Vertical/Horizontal -->
-   <!-- Orientation seem to be correct -->
-  <xacro:mil_thruster
-    name="FLV"
-    parent="base_link"
-    xyz="-0.15217 -0.16474 0.010449"
-    rpy="0 0 0"
-  />
-  <xacro:mil_thruster
-    name="FRV"
-    parent="base_link"
-    xyz="-0.1492 0.13821 0.010449"
-    rpy="0 0 0"
-  />
-  <xacro:mil_thruster
-    name="BRV"
-    parent="base_link"
-    xyz="0.31117 0.13821 0.010449"
-    rpy="0 0 0"
-  />
-  <xacro:mil_thruster
-    name="BLV"
-    parent="base_link"
-    xyz="0.30868 -0.16621 0.010449"
-    rpy="0 0 0"
-  />
-  <xacro:mil_thruster
-    name="FLH"
-    parent="base_link"
-    xyz="-0.14714 -0.26409 0.038317"
-    rpy="-1.5708 0 0.7854"
-  />
-  <xacro:mil_thruster
-    name="FRH"
-    parent="base_link"
-    xyz="-0.147 0.2413 0.038324"
-    rpy="1.5708 0 -0.7854"
-  />
-  <xacro:mil_thruster
-    name="BRH"
-    parent="base_link"
-    xyz="0.32369 0.22645 0.038317"
-    rpy="-1.5708 0 0.7854"
-  />
-  <xacro:mil_thruster
-    name="BLH"
-    parent="base_link"
-    xyz="0.32397 -0.25204 0.038324"
-    rpy="1.5708 0 -0.7854"
-  />
+  <!-- Thrusters -->
+  <!-- Front/Back Left/Right Vertical/Horizontal -->
+  <!-- Orientation seem to be correct -->
+  <xacro:mil_thruster name="FLV" parent="base_link" xyz="-0.15217 -0.16474 0.010449" rpy="0 0 0"/>
+  <xacro:mil_thruster name="FRV" parent="base_link" xyz="-0.1492 0.13821 0.010449" rpy="0 0 0"/>
+  <xacro:mil_thruster name="BRV" parent="base_link" xyz="0.31117 0.13821 0.010449" rpy="0 0 0"/>
+  <xacro:mil_thruster name="BLV" parent="base_link" xyz="0.30868 -0.16621 0.010449" rpy="0 0 0"/>
+  <xacro:mil_thruster name="FLH" parent="base_link" xyz="-0.14714 -0.26409 0.038317" rpy="-1.5708 0 0.7854"/>
+  <xacro:mil_thruster name="FRH" parent="base_link" xyz="-0.147 0.2413 0.038324" rpy="1.5708 0 -0.7854"/>
+  <xacro:mil_thruster name="BRH" parent="base_link" xyz="0.32369 0.22645 0.038317" rpy="-1.5708 0 0.7854"/>
+  <xacro:mil_thruster name="BLH" parent="base_link" xyz="0.32397 -0.25204 0.038324" rpy="1.5708 0 -0.7854"/>
 </robot>

File: src/subjugator/simulation/subjugator_description/urdf/xacro/camera.xacro (robot description, xacro)
@@ -2,12 +2,9 @@
 <robot xmlns:xacro="http://ros.org/wiki/xacro">
   <!-- Macro for inserting a camera -->
-  <xacro:macro
-    name="mil_camera"
-    params="name parent xyz rpy
+  <xacro:macro name="mil_camera" params="name parent xyz rpy
             use_image_processing=false
-            width=960 height=600 fov=1.047 fps=30"
-  >
+            width=960 height=600 fov=1.047 fps=30">
     <!-- Camera Link -->
-     <link name="${name}_link">
+    <link name="${name}_link">
       <origin xyz="0 0 0" rpy="0 0 0"/>
       <inertial>
@@ -46,7 +43,5 @@
         </camera>
         <xacro:if value="${use_image_processing}">
-          <plugin
-            filename="UnderwaterCamera"
-            name="dave_gz_sensor_plugins::UnderwaterCamera">
+          <plugin filename="UnderwaterCamera" name="dave_gz_sensor_plugins::UnderwaterCamera">
             <attenuationR>0.8</attenuationR>
             <attenuationG>0.5</attenuationG>

File: src/subjugator/simulation/subjugator_description/urdf/xacro/dvl.xacro (robot description, xacro)
@@ -2,10 +2,7 @@
 <robot xmlns:xacro="http://ros.org/wiki/xacro" xmlns:experimental="http://sdformat.org/schemas/experimental" xmlns:gz="http://gazebosim.org/schema">
   <!-- Macro for inserting a DVL -->
-  <xacro:macro
-    name="mil_dvl_sensor"
-    params="name parent xyz rpy"
-  >
+  <xacro:macro name="mil_dvl_sensor" params="name parent xyz rpy">
     <!-- DVL Link -->
-     <link name="${name}_link">
+    <link name="${name}_link">
       <origin xyz="0 0 0" rpy="0 0 0"/>
       <inertial>
@@ -28,7 +25,5 @@
     <!-- Sensor/Plugin Info-->
     <gazebo reference="${name}_link">
-      <sensor
-        name="A50_Waterlinked" type="custom"
-        gz:type="dvl">
+      <sensor name="A50_Waterlinked" type="custom" gz:type="dvl">
         <pose>0 0 0 0 0 0</pose>
         <always_on>1</always_on>
@@ -93,11 +88,9 @@
     </gazebo>
     <gazebo>
-        <plugin
-          filename="DVLBridge"
-          name="dave_ros_gz_plugins::DVLBridge">
-          <!-- Grabbed in DVL Bridge script -->
-          <topic>/dvl/velocity</topic>
-        </plugin>
-      </gazebo>
-    </xacro:macro>
+      <plugin filename="DVLBridge" name="dave_ros_gz_plugins::DVLBridge">
+        <!-- Grabbed in DVL Bridge script -->
+        <topic>/dvl/velocity</topic>
+      </plugin>
+    </gazebo>
+  </xacro:macro>
 </robot>

File: src/subjugator/simulation/subjugator_description/urdf/xacro/fixed_link.xacro (robot description, xacro)
@@ -1,5 +1,5 @@
 <?xml version="1.0"?>
 <robot xmlns:xacro="http://ros.org/wiki/xacro">
-<!-- Macro to allow the quick creation of a fixed link-->
+  <!-- Macro to allow the quick creation of a fixed link-->
   <xacro:macro name="mil_fixed_link" params="name parent='base_link'
                         xyz:='0 0 0' rpy:='0 0 0'">

File: src/subjugator/simulation/subjugator_description/urdf/xacro/imu_magnetometer.xacro (robot description, xacro)
@@ -1,11 +1,8 @@
 <?xml version="1.0"?>
 <robot xmlns:xacro="http://ros.org/wiki/xacro">
-  <xacro:macro
-    name="mil_imu_magnetometer"
-    params="name namespace parent xyz rpy
-            rate ax ay az lx ly lz"
-  >
-   <!-- Imu link -->
-   <link name="${name}_link">
+  <xacro:macro name="mil_imu_magnetometer" params="name namespace parent xyz rpy
+            rate ax ay az lx ly lz">
+    <!-- Imu link -->
+    <link name="${name}_link">
       <origin xyz="0 0 0" rpy="0 0 0"/>
       <inertial>
@@ -28,8 +25,9 @@
     <!-- Sensor/Plugin Info-->
     <gazebo reference="${name}_link">
-      <sensor name="VectorNav_IMU" type="imu">
+      <sensor name="${name}_link" type="imu">
         <always_on>true</always_on>
         <update_rate>${rate}</update_rate>
         <topic>${namespace}/data_raw</topic>
+        <gz_frame_id>imu_link</gz_frame_id>
         <imu>
           <linear_acceleration>
@@ -68,8 +66,5 @@
           </angular_velocity>
         </imu>
-        <plugin
-            filename="gz-sim-imu-system"
-            name="gz::sim::systems::Imu">
-        </plugin>
+        <plugin filename="gz-sim-imu-system" name="gz::sim::systems::Imu"/>
       </sensor>
       <sensor name="VectorNav_MAG" type="magnetometer">
@@ -77,10 +72,7 @@
         <update_rate>${rate}</update_rate>
         <topic>${namespace}/mag</topic>
-        <plugin
-            filename="gz-sim-magnetometer-system"
-            name="gz::sim::systems::Magnetometer">
-        </plugin>
+        <plugin filename="gz-sim-magnetometer-system" name="gz::sim::systems::Magnetometer"/>
       </sensor>
     </gazebo>
-    </xacro:macro>
+  </xacro:macro>
 </robot>

File: src/subjugator/simulation/subjugator_description/urdf/xacro/thruster.xacro (robot description, xacro)
@@ -2,9 +2,7 @@
 <robot xmlns:xacro="http://www.ros.org/wiki/xacro">
   <!-- Macro for inserting a Thruster -->
-  <xacro:macro
-    name="mil_thruster"
-    params="name parent xyz rpy">
+  <xacro:macro name="mil_thruster" params="name parent xyz rpy">
     <!-- Link for base of thruster (this is for TF) -->
-     <link name="${name}_link">
+    <link name="${name}_link">
       <origin xyz="0 0 0" rpy="0 0 0"/>
       <inertial>
@@ -47,7 +45,5 @@
     <!-- Don't give it a reference like the other plugins-->
     <gazebo>
-      <plugin
-        filename="gz-sim-thruster-system"
-        name="gz::sim::systems::Thruster">
+      <plugin filename="gz-sim-thruster-system" name="gz::sim::systems::Thruster">
         <namespace>${name}</namespace>
         <use_angvel_cmd>0</use_angvel_cmd>

Commit message: ran pre-commit

File: src/subjugator/simulation/subjugator_description/urdf/sub9.urdf.xacro (robot description, xacro)
@@ -80,16 +80,6 @@
     lz="0.08825985"
   />
-   <!--Depth Sensor-->
-  <xacro:mil_depth_sensor
-    name="depth_sensor"
-    namespace="/depth"
-    parent="base_link"
-    xyz="0 0 0"
-    rpy="0 0 0"
-    update_rate="5"
-    frame_id="depth_sensor_frame"
-    noise_mean="0.0"
-    noise_stddev="0"
-  />
+  <!--Depth Sensor-->
+  <xacro:mil_depth_sensor name="depth_sensor" namespace="/depth" parent="base_link" xyz="0 0 0" rpy="0 0 0" update_rate="5" frame_id="depth_sensor_frame" noise_mean="0.0" noise_stddev="0"/>
   <!-- Thrusters -->
   <!-- Front/Back Left/Right Vertical/Horizontal -->

File: src/subjugator/simulation/subjugator_description/urdf/xacro/depth.xacro (robot description, xacro)
@@ -16,10 +16,10 @@
   >
     <link name="${name}_link">
+      <origin xyz="0 0 0" rpy="0 0 0"/>
+      <inertial>
         <origin xyz="0 0 0" rpy="0 0 0"/>
-        <inertial>
-            <origin xyz="0 0 0" rpy="0 0 0"/>
-            <mass value="0.1"/>
-            <inertia ixx="0.001" iyy="0.001" izz="0.001" ixy="0" ixz="0" iyz="0"/>
-        </inertial>
+        <mass value="0.1"/>
+        <inertia ixx="0.001" iyy="0.001" izz="0.001" ixy="0" ixz="0" iyz="0"/>
+      </inertial>
     </link>
     <!-- DepthSensor Joint -->
@@ -34,14 +34,14 @@
       <preserveFixedJoint>true</preserveFixedJoint>
     </gazebo>
-    <gazebo >
-        <plugin name="depth_sensor::DepthSensor" filename="DepthSensor">
-            <!-- SDF parameters -->
-            <frame_id>${frame_id}</frame_id>
-            <offset>0 0 0 0 0 0</offset>
-            <topic>/depth</topic>
-            <update_rate>${update_rate}</update_rate>
-            <noise_mean>${noise_mean}</noise_mean>
-            <noise_stddev>${noise_stddev}</noise_stddev>
-        </plugin>
+    <gazebo>
+      <plugin name="depth_sensor::DepthSensor" filename="DepthSensor">
+        <!-- SDF parameters -->
+        <frame_id>${frame_id}</frame_id>
+        <offset>0 0 0 0 0 0</offset>
+        <topic>/depth</topic>
+        <update_rate>${update_rate}</update_rate>
+        <noise_mean>${noise_mean}</noise_mean>
+        <noise_stddev>${noise_stddev}</noise_stddev>
+      </plugin>
     </gazebo>
   </xacro:macro>

Commit message: Fixed URDF thruster locations

File: src/subjugator/simulation/subjugator_description/urdf/sub9.urdf.xacro (robot description, xacro)
@@ -12,5 +12,5 @@
   <link name="base_link">
     <!-- Sub's Pose -->
-    <origin rpy="0 0 0" xyz="-0.1 0.0125 -1"/>
+    <origin rpy="0 0 0" xyz="0 0 0"/>
     <!-- Inertial Properties -->
     <inertial>
@@ -22,5 +22,5 @@
     <!-- Visual Data-->
     <visual name="visual">
-      <origin rpy="0 0 0" xyz="0 0 0"/>
+      <origin rpy="0 0 0" xyz="-0.254 0 0"/>
       <geometry>
         <mesh filename="package://subjugator_description/urdf/meshes/Sub9.dae"/>
@@ -85,11 +85,11 @@
   <!-- Front/Back Left/Right Vertical/Horizontal -->
   <!-- Orientation seem to be correct -->
-  <xacro:mil_thruster name="FLV" parent="base_link" xyz="-0.15217 -0.16474 0.010449" rpy="0 0 0"/>
-  <xacro:mil_thruster name="FRV" parent="base_link" xyz="-0.1492 0.13821 0.010449" rpy="0 0 0"/>
-  <xacro:mil_thruster name="BRV" parent="base_link" xyz="0.31117 0.13821 0.010449" rpy="0 0 0"/>
-  <xacro:mil_thruster name="BLV" parent="base_link" xyz="0.30868 -0.16621 0.010449" rpy="0 0 0"/>
-  <xacro:mil_thruster name="FLH" parent="base_link" xyz="-0.14714 -0.26409 0.038317" rpy="-1.5708 0 0.7854"/>
-  <xacro:mil_thruster name="FRH" parent="base_link" xyz="-0.147 0.2413 0.038324" rpy="1.5708 0 -0.7854"/>
-  <xacro:mil_thruster name="BRH" parent="base_link" xyz="0.32369 0.22645 0.038317" rpy="-1.5708 0 0.7854"/>
-  <xacro:mil_thruster name="BLH" parent="base_link" xyz="0.32397 -0.25204 0.038324" rpy="1.5708 0 -0.7854"/>
+  <xacro:mil_thruster name="FLV" parent="base_link" xyz="0.3175 0.14922 -0.028575" rpy="0 -1.57079 0"/>
+  <xacro:mil_thruster name="FRV" parent="base_link" xyz="0.3175 -0.14922 -0.02875" rpy="0 -1.57079 0"/>
+  <xacro:mil_thruster name="BRV" parent="base_link" xyz="-0.1307 -0.14922 -0.028575" rpy="0 -1.57079 0"/>
+  <xacro:mil_thruster name="BLV" parent="base_link" xyz="-0.1307 0.14922 -0.028575" rpy="0 -1.57079 0"/>
+  <xacro:mil_thruster name="FLH" parent="base_link" xyz="0.33337 0.24765 0.053875" rpy="0 0 5.72468"/>
+  <xacro:mil_thruster name="FRH" parent="base_link" xyz="0.33337 -0.24765 0.053975" rpy="0 0 -5.72468"/>
+  <xacro:mil_thruster name="BRH" parent="base_link" xyz="-0.127 -0.24765 0.049213" rpy="0 0 -1.01229"/>
+  <xacro:mil_thruster name="BLH" parent="base_link" xyz="-0.127 0.24765 0.053975" rpy="0 0 1.01229"/>
 </robot>

Commit message: Tweak thruster locations and rotations

File: src/subjugator/simulation/subjugator_description/urdf/sub9.urdf.xacro (robot description, xacro)
@@ -8,9 +8,8 @@
   <xacro:include filename="$(find subjugator_description)/urdf/xacro/collision.xacro"/>
   <xacro:include filename="$(find subjugator_description)/urdf/xacro/thruster.xacro"/>
-  <xacro:include filename="$(find subjugator_description)/urdf/xacro/depth.xacro"/>
   <!-- Base Link of the Sub -->
   <link name="base_link">
     <!-- Sub's Pose -->
-    <origin rpy="0 0 0" xyz="0 0 0"/>
+    <origin rpy="0 0 0" xyz="-0.1 0.0125 -1"/>
     <!-- Inertial Properties -->
     <inertial>
@@ -22,5 +21,5 @@
     <!-- Visual Data-->
     <visual name="visual">
-      <origin rpy="0 0 0" xyz="-0.254 0 0"/>
+      <origin rpy="0 0 3.1415" xyz="0 0 0"/>
       <geometry>
         <mesh filename="package://subjugator_description/urdf/meshes/Sub9.dae"/>
@@ -80,16 +79,14 @@
     lz="0.08825985"
   />
-  <!--Depth Sensor-->
-  <xacro:mil_depth_sensor name="depth_sensor" namespace="/depth" parent="base_link" xyz="0 0 0" rpy="0 0 0" update_rate="5" frame_id="depth_sensor_frame" noise_mean="0.0" noise_stddev="0"/>
   <!-- Thrusters -->
   <!-- Front/Back Left/Right Vertical/Horizontal -->
   <!-- Orientation seem to be correct -->
-  <xacro:mil_thruster name="FLV" parent="base_link" xyz="0.3175 0.14922 -0.028575" rpy="0 -1.57079 0"/>
-  <xacro:mil_thruster name="FRV" parent="base_link" xyz="0.3175 -0.14922 -0.02875" rpy="0 -1.57079 0"/>
-  <xacro:mil_thruster name="BRV" parent="base_link" xyz="-0.1307 -0.14922 -0.028575" rpy="0 -1.57079 0"/>
-  <xacro:mil_thruster name="BLV" parent="base_link" xyz="-0.1307 0.14922 -0.028575" rpy="0 -1.57079 0"/>
-  <xacro:mil_thruster name="FLH" parent="base_link" xyz="0.33337 0.24765 0.053875" rpy="0 0 5.72468"/>
-  <xacro:mil_thruster name="FRH" parent="base_link" xyz="0.33337 -0.24765 0.053975" rpy="0 0 -5.72468"/>
-  <xacro:mil_thruster name="BRH" parent="base_link" xyz="-0.127 -0.24765 0.049213" rpy="0 0 -1.01229"/>
-  <xacro:mil_thruster name="BLH" parent="base_link" xyz="-0.127 0.24765 0.053975" rpy="0 0 1.01229"/>
+  <xacro:mil_thruster name="FLV" parent="base_link" xyz="-0.40617 -0.16474 0.010449" rpy="0 -1.5708 0"/>
+  <xacro:mil_thruster name="FRV" parent="base_link" xyz="-0.4032 0.13821 0.010449" rpy="0 -1.5708 0"/>
+  <xacro:mil_thruster name="BRV" parent="base_link" xyz="0.05717 0.13821 0.010449" rpy="0 -1.5708 0"/>
+  <xacro:mil_thruster name="BLV" parent="base_link" xyz="0.05468 -0.16621 0.010449" rpy="0 -1.5708 0"/>
+  <xacro:mil_thruster name="FLH" parent="base_link" xyz="-0.40114 -0.26409 0.038317" rpy="0 0 0"/>
+  <xacro:mil_thruster name="FRH" parent="base_link" xyz="-0.401 0.2413 0.038324" rpy="0 0 0"/>
+  <xacro:mil_thruster name="BRH" parent="base_link" xyz="0.06969 0.22645 0.038317" rpy="0 0 0"/>
+  <xacro:mil_thruster name="BLH" parent="base_link" xyz="0.06997 -0.25204 0.038324" rpy="0 0 0"/>
 </robot>

File: src/subjugator/simulation/subjugator_description/urdf/xacro/thruster.xacro (robot description, xacro)
@@ -35,9 +35,8 @@
     <!-- Thruster Direction joint -->
     <joint name="${name}_dir_joint" type="revolute">
-      <origin xyz="0 0 1" rpy="0 0 0"/>
+      <origin xyz="0 0 0" rpy="0 0"/>
       <parent link="${name}_link"/>
       <child link="${name}_dir_link"/>
       <limit effort="1000" lower="0.0" upper="0.548" velocity="0.5"/>
-      <axis xyz="0 0 1"/>
     </joint>
     <!-- Sensor/Plugin Info-->

Commit message: Re-add depth sensor that was lost in previous commit

File: src/subjugator/simulation/subjugator_description/urdf/sub9.urdf.xacro (robot description, xacro)
@@ -8,4 +8,5 @@
   <xacro:include filename="$(find subjugator_description)/urdf/xacro/collision.xacro"/>
   <xacro:include filename="$(find subjugator_description)/urdf/xacro/thruster.xacro"/>
+  <xacro:include filename="$(find subjugator_description)/urdf/xacro/depth.xacro"/>
   <!-- Base Link of the Sub -->
   <link name="base_link">
@@ -79,4 +80,16 @@
     lz="0.08825985"
   />
+  <!--Depth Sensor-->
+  <xacro:mil_depth_sensor
+    name="depth_sensor"
+    namespace="/depth"
+    parent="base_link"
+    xyz="0 0 0"
+    rpy="0 0 0"
+    update_rate="5"
+    frame_id="depth_sensor_frame"
+    noise_mean="0.0"
+    noise_stddev="0"
+  />
   <!-- Thrusters -->
   <!-- Front/Back Left/Right Vertical/Horizontal -->

File: src/subjugator/simulation/subjugator_description/urdf/xacro/thruster.xacro (robot description, xacro)
@@ -35,5 +35,5 @@
     <!-- Thruster Direction joint -->
     <joint name="${name}_dir_joint" type="revolute">
-      <origin xyz="0 0 0" rpy="0 0"/>
+      <origin xyz="0 0 0" rpy="0 0 0"/>
       <parent link="${name}_link"/>
       <child link="${name}_dir_link"/>
