Commit message: Re-add depth sensor that was lost in previous commit

File: src/subjugator/simulation/subjugator_description/urdf/sub9.urdf.xacro (robot description, xacro)
@@ -12,15 +12,15 @@
   <link name="base_link">
     <!-- Sub's Pose -->
-    <origin rpy="0 0 0" xyz="-0.1 0.0125 -1"/>
+    <origin rpy="0 0 0" xyz="0 0 0"/>
     <!-- Inertial Properties -->
     <inertial>
-      <origin rpy="0 0 0" xyz="0 0 0"/>
+      <origin rpy="0 0 0" xyz="0.254 0 0"/>
       <!-- Need to be properly calculated at some point -->
-      <mass value="30.5"/>
-      <inertia ixx="0.96105" ixy="0.003" ixz="-0.02" iyy="1.799" iyz="0.0003" izz="2.1286"/>
+      <mass value="60.5"/>
+      <inertia ixx="0.4831007" ixy="0.0043714" ixz="-0.2404290" iyy="2.7671192" iyz="-0.0043714" izz="2.2993755"/>
     </inertial>
     <!-- Visual Data-->
     <visual name="visual">
-      <origin rpy="0 0 3.1415" xyz="0 0 0"/>
+      <origin rpy="0 0 0" xyz="0 0 0"/>
       <geometry>
         <mesh filename="package://subjugator_description/urdf/meshes/Sub9.dae"/>
@@ -30,5 +30,5 @@
     <collision name="main_collision">
       <!-- This collision is for calculating the buoyant forces-->
-      <origin rpy="0 0 0" xyz="0 0 0.1"/>
+      <origin rpy="0 0 0" xyz="0.254 0 0"/>
       <geometry>
         <box size="0.9 0.35 0.2"/>
@@ -61,23 +61,35 @@
   </gazebo>
   <!-- Cameras -->
-  <xacro:mil_camera name="front_cam" parent="base_link" xyz="-0.32 -0.014274 -0.050" rpy="0 0 3.14159"/>
-  <xacro:mil_camera name="down_cam" parent="base_link" xyz="-0.15222 0.027913 -0.22" rpy="0 1.57 0"/>
+  <!-- <xacro:mil_camera name="front_cam" parent="base_link" xyz="-0.32 -0.014274 -0.050" rpy="0 0 3.14159"/> -->
+  <!-- <xacro:mil_camera name="down_cam" parent="base_link" xyz="-0.15222 0.027913 -0.22" rpy="0 1.57 0"/> -->
   <!-- DVL Sensor -->
-  <xacro:mil_dvl_sensor name="dvl_sensor" parent="base_link" xyz="0.21236 0.00254 -0.10233" rpy="0 0 0"/>
+  <!-- <xacro:mil_dvl_sensor name="dvl_sensor" parent="base_link" xyz="0.21236 0.00254 -0.10233" rpy="0 0 0"/> -->
   <!-- IMU, Magnetometer -->
-  <xacro:mil_imu_magnetometer
-    name="imu"
-    namespace='/imu'
-    parent="base_link"
-    xyz="0.0632 -0.164 -0.079"
-    rpy="0 0 0"
-    rate="210"
-    ax="0.015707963"
-    ay="0.015707963"
-    az="0.015707963"
-    lx="0.08825985"
-    ly="0.08825985"
-    lz="0.08825985"
-  />
+  <!-- <xacro:mil_imu_magnetometer -->
+  <!--   name="imu" -->
+  <!--   namespace='/imu' -->
+  <!--   parent="base_link" -->
+  <!--   xyz="0.0632 -0.164 -0.079" -->
+  <!--   rpy="0 0 0" -->
+  <!--   rate="210" -->
+  <!--   ax="0.015707963" -->
+  <!--   ay="0.015707963" -->
+  <!--   az="0.015707963" -->
+  <!--   lx="0.08825985" -->
+  <!--   ly="0.08825985" -->
+  <!--   lz="0.08825985" -->
+  <!-- /> -->
+  <!--Depth Sensor-->
+  <!-- <xacro:mil_depth_sensor  -->
+  <!--   name="depth_sensor" -->
+  <!--   namespace="/depth" -->
+  <!--   parent="base_link"  -->
+  <!--   xyz="0 0 0"  -->
+  <!--   rpy="0 0 0"  -->
+  <!--   update_rate="5"  -->
+  <!--   frame_id="depth_sensor_frame"  -->
+  <!--   noise_mean="0.0"  -->
+  <!--   noise_stddev="0" -->
+  <!-- /> -->
   <!--Depth Sensor-->
   <xacro:mil_depth_sensor
@@ -95,11 +107,11 @@
   <!-- Front/Back Left/Right Vertical/Horizontal -->
   <!-- Orientation seem to be correct -->
-  <xacro:mil_thruster name="FLV" parent="base_link" xyz="-0.40617 -0.16474 0.010449" rpy="0 -1.5708 0"/>
-  <xacro:mil_thruster name="FRV" parent="base_link" xyz="-0.4032 0.13821 0.010449" rpy="0 -1.5708 0"/>
-  <xacro:mil_thruster name="BRV" parent="base_link" xyz="0.05717 0.13821 0.010449" rpy="0 -1.5708 0"/>
-  <xacro:mil_thruster name="BLV" parent="base_link" xyz="0.05468 -0.16621 0.010449" rpy="0 -1.5708 0"/>
-  <xacro:mil_thruster name="FLH" parent="base_link" xyz="-0.40114 -0.26409 0.038317" rpy="0 0 0"/>
-  <xacro:mil_thruster name="FRH" parent="base_link" xyz="-0.401 0.2413 0.038324" rpy="0 0 0"/>
-  <xacro:mil_thruster name="BRH" parent="base_link" xyz="0.06969 0.22645 0.038317" rpy="0 0 0"/>
-  <xacro:mil_thruster name="BLH" parent="base_link" xyz="0.06997 -0.25204 0.038324" rpy="0 0 0"/>
+  <xacro:mil_thruster name="FLV" parent="base_link" xyz="0.5715 0.14922 -0.028575" rpy="0 -1.5708 0"/>
+  <xacro:mil_thruster name="FRV" parent="base_link" xyz="0.5715 -0.14922 -0.028575" rpy="0 -1.5708 0"/>
+  <xacro:mil_thruster name="BRV" parent="base_link" xyz="0.1143 -0.14922 -0.028575" rpy="0 -1.5708 0"/>
+  <xacro:mil_thruster name="BLV" parent="base_link" xyz="0.1143 0.14922 -0.028575" rpy="0 -1.5708 0"/>
+  <xacro:mil_thruster name="FLH" parent="base_link" xyz="0.58737 0.24765 0.053975" rpy="0 0 5.72468"/>
+  <xacro:mil_thruster name="FRH" parent="base_link" xyz="0.58737 -0.24765 0.053975" rpy="0 0 -5.72468"/>
+  <xacro:mil_thruster name="BRH" parent="base_link" xyz="0.127 -0.24765 0.053975" rpy="0 0 -1.01229"/>
+  <xacro:mil_thruster name="BLH" parent="base_link" xyz="0.127 0.24765 0.053975" rpy="0 0 1.01229"/>
 </robot>

Commit message: Fixed sub inertials

File: src/subjugator/simulation/subjugator_description/urdf/sub9.urdf.xacro (robot description, xacro)
@@ -15,8 +15,8 @@
     <!-- Inertial Properties -->
     <inertial>
-      <origin rpy="0 0 0" xyz="0.254 0 0"/>
+      <origin rpy="0 0 0" xyz="0.354 0 0"/>
       <!-- Need to be properly calculated at some point -->
-      <mass value="60.5"/>
-      <inertia ixx="0.4831007" ixy="0.0043714" ixz="-0.2404290" iyy="2.7671192" iyz="-0.0043714" izz="2.2993755"/>
+      <mass value="22.5"/>
+      <inertia ixx="2.4" ixy="0" ixz="0" iyy="2.4" iyz="0.0" izz="3.0"/>
     </inertial>
     <!-- Visual Data-->
@@ -28,22 +28,53 @@
     </visual>
     <!-- Collision Data -->
-    <collision name="main_collision">
+    <collision name="buoyancy_collision">
       <!-- This collision is for calculating the buoyant forces-->
-      <origin rpy="0 0 0" xyz="0.254 0 0"/>
+      <origin rpy="0 0 0" xyz="0.354 0 0"/>
       <geometry>
-        <box size="0.9 0.35 0.2"/>
+        <sphere radius="0.1725"/>
       </geometry>
     </collision>
-    <!-- Need to add 'shell' collisions-->
+    <!-- The following are shell collisions. They dont contrubute to buoyancy-->
+    <!-- and are for collisions -->
+    <collision name="Front_Shell">
+      <origin rpy="0 0 0" xyz="0.708 0 0"/>
+      <geometry>
+        <box size="0.001 0.345 0.345"/>
+      </geometry>
+    </collision>
+    <collision name="Back_Shell">
+      <origin rpy="0 0 0" xyz="0 0 0"/>
+      <geometry>
+        <box size="0.001 0.345 0.345"/>
+      </geometry>
+    </collision>
+    <collision name="Left_Shell">
+      <origin rpy="0 0 0" xyz="0.345 0.177 0"/>
+      <geometry>
+        <box size="0.708 0.001 0.345"/>
+      </geometry>
+    </collision>
+    <collision name="Right_Shell">
+      <origin rpy="0 0 0" xyz="0.345 -0.177 0"/>
+      <geometry>
+        <box size="0.708 0.001 0.345"/>
+      </geometry>
+    </collision>
+    <collision name="Top_Shell">
+      <origin rpy="0 0 0" xyz="0.345 0 0.177"/>
+      <geometry>
+        <box size="0.708 0.345 0.001"/>
+      </geometry>
+    </collision>
+    <collision name="Front_Shell">
+      <origin rpy="0 0 0" xyz="0.345 0 -0.177"/>
+      <geometry>
+        <box size="0.708 0.345 0.001"/>
+      </geometry>
+    </collision>
   </link>
   <gazebo>
     <plugin filename="gz-sim-hydrodynamics-system" name="gz::sim::systems::Hydrodynamics">
       <link_name>base_link</link_name>
-      <xDotU>-2</xDotU>
-      <yDotV>-5</yDotV>
-      <zDotW>-5</zDotW>
-      <kDotP>-0.1</kDotP>
-      <mDotQ>-1</mDotQ>
-      <nDotR>-1</nDotR>
       <xUabsU>-25</xUabsU>
       <xU>-50</xU>
@@ -52,59 +83,36 @@
       <zWabsW>-5</zWabsW>
       <zW>-50</zW>
-      <kPabsP>-5</kPabsP>
-      <kP>-10</kP>
-      <mQabsQ>-5</mQabsQ>
-      <mQ>-10</mQ>
-      <nRabsR>-5</nRabsR>
-      <nR>-10</nR>
+      <kPabsP>-650</kPabsP>
+      <kP>-650</kP>
+      <mQabsQ>-750</mQabsQ>
+      <mQ>-750</mQ>
+      <nRabsR>-750</nRabsR>
+      <nR>-750</nR>
     </plugin>
   </gazebo>
   <!-- Cameras -->
-  <!-- <xacro:mil_camera name="front_cam" parent="base_link" xyz="-0.32 -0.014274 -0.050" rpy="0 0 3.14159"/> -->
-  <!-- <xacro:mil_camera name="down_cam" parent="base_link" xyz="-0.15222 0.027913 -0.22" rpy="0 1.57 0"/> -->
+  <xacro:mil_camera name="front_cam" parent="base_link" xyz="0.78 -0.014274 -0.050" rpy="0 0 0"/>
+  <xacro:mil_camera name="down_cam" parent="base_link" xyz="0.45222 0.027913 -0.22" rpy="0 1.57 0"/>
   <!-- DVL Sensor -->
-  <!-- <xacro:mil_dvl_sensor name="dvl_sensor" parent="base_link" xyz="0.21236 0.00254 -0.10233" rpy="0 0 0"/> -->
+  <xacro:mil_dvl_sensor name="dvl_sensor" parent="base_link" xyz="0.41236 0.00254 -0.10233" rpy="0 0 0"/>
   <!-- IMU, Magnetometer -->
-  <!-- <xacro:mil_imu_magnetometer -->
-  <!--   name="imu" -->
-  <!--   namespace='/imu' -->
-  <!--   parent="base_link" -->
-  <!--   xyz="0.0632 -0.164 -0.079" -->
-  <!--   rpy="0 0 0" -->
-  <!--   rate="210" -->
-  <!--   ax="0.015707963" -->
-  <!--   ay="0.015707963" -->
-  <!--   az="0.015707963" -->
-  <!--   lx="0.08825985" -->
-  <!--   ly="0.08825985" -->
-  <!--   lz="0.08825985" -->
-  <!-- /> -->
+  <xacro:mil_imu_magnetometer
+    name="imu"
+    namespace='/imu'
+    parent="base_link"
+    xyz="0.3632 -0.164 -0.079"
+    rpy="0 0 0"
+    rate="210"
+    ax="0.015707963"
+    ay="0.015707963"
+    az="0.015707963"
+    lx="0.08825985"
+    ly="0.08825985"
+    lz="0.08825985"
+  />
   <!--Depth Sensor-->
-  <!-- <xacro:mil_depth_sensor  -->
-  <!--   name="depth_sensor" -->
-  <!--   namespace="/depth" -->
-  <!--   parent="base_link"  -->
-  <!--   xyz="0 0 0"  -->
-  <!--   rpy="0 0 0"  -->
-  <!--   update_rate="5"  -->
-  <!--   frame_id="depth_sensor_frame"  -->
-  <!--   noise_mean="0.0"  -->
-  <!--   noise_stddev="0" -->
-  <!-- /> -->
-  <!--Depth Sensor-->
-  <xacro:mil_depth_sensor
-    name="depth_sensor"
-    namespace="/depth"
-    parent="base_link"
-    xyz="0 0 0"
-    rpy="0 0 0"
-    update_rate="5"
-    frame_id="depth_sensor_frame"
-    noise_mean="0.0"
-    noise_stddev="0"
-  />
+  <xacro:mil_depth_sensor name="depth_sensor" namespace="/depth" parent="base_link" xyz="0.3 0 0" rpy="0 0 0" update_rate="5" frame_id="depth_sensor_frame" noise_mean="0.0" noise_stddev="0"/>
   <!-- Thrusters -->
   <!-- Front/Back Left/Right Vertical/Horizontal -->
-  <!-- Orientation seem to be correct -->
   <xacro:mil_thruster name="FLV" parent="base_link" xyz="0.5715 0.14922 -0.028575" rpy="0 -1.5708 0"/>
   <xacro:mil_thruster name="FRV" parent="base_link" xyz="0.5715 -0.14922 -0.028575" rpy="0 -1.5708 0"/>

Commit message: Thruster manager and urdf updates (#83)
* thruster_manager: now uses parameters and new custom msg output type

* subjugator_msgs: removed unused thruster related msgs and srvs

* Made tam more realistic, updated topic names

* prototype for connecting to sim (only vert thrusters)

* Fixed URDF thruster locations

* better thruster mapper, loops, more real matrix

* added simulation connection to launch, renamed things

* Tweak thruster locations and rotations

* Re-add depth sensor that was lost in previous commit

* Re-add depth sensor that was lost in previous commit

* real math, 30 deg angle

* Fixed sub inertials

* fixed urdf angles, added thruster manager to general launch

* updated blender file for angles

* fixed precommit thruster manager

* made header file for thruster mapper

* added pragma once

---------

Co-authored-by: keith khadar <keith.khadar@gmail.com>
Co-authored-by: oixel <oycell@aol.com>

File: src/subjugator/simulation/subjugator_description/urdf/sub9.urdf.xacro (robot description, xacro)
@@ -12,11 +12,11 @@
   <link name="base_link">
     <!-- Sub's Pose -->
-    <origin rpy="0 0 0" xyz="-0.1 0.0125 -1"/>
+    <origin rpy="0 0 0" xyz="0 0 0"/>
     <!-- Inertial Properties -->
     <inertial>
-      <origin rpy="0 0 0" xyz="0 0 0"/>
+      <origin rpy="0 0 0" xyz="0.354 0 0"/>
       <!-- Need to be properly calculated at some point -->
-      <mass value="30.5"/>
-      <inertia ixx="0.96105" ixy="0.003" ixz="-0.02" iyy="1.799" iyz="0.0003" izz="2.1286"/>
+      <mass value="22.5"/>
+      <inertia ixx="2.4" ixy="0" ixz="0" iyy="2.4" iyz="0.0" izz="3.0"/>
     </inertial>
     <!-- Visual Data-->
@@ -28,22 +28,53 @@
     </visual>
     <!-- Collision Data -->
-    <collision name="main_collision">
+    <collision name="buoyancy_collision">
       <!-- This collision is for calculating the buoyant forces-->
-      <origin rpy="0 0 0" xyz="0 0 0.1"/>
+      <origin rpy="0 0 0" xyz="0.354 0 0"/>
       <geometry>
-        <box size="0.9 0.35 0.2"/>
+        <sphere radius="0.1725"/>
       </geometry>
     </collision>
-    <!-- Need to add 'shell' collisions-->
+    <!-- The following are shell collisions. They dont contrubute to buoyancy-->
+    <!-- and are for collisions -->
+    <collision name="Front_Shell">
+      <origin rpy="0 0 0" xyz="0.708 0 0"/>
+      <geometry>
+        <box size="0.001 0.345 0.345"/>
+      </geometry>
+    </collision>
+    <collision name="Back_Shell">
+      <origin rpy="0 0 0" xyz="0 0 0"/>
+      <geometry>
+        <box size="0.001 0.345 0.345"/>
+      </geometry>
+    </collision>
+    <collision name="Left_Shell">
+      <origin rpy="0 0 0" xyz="0.345 0.177 0"/>
+      <geometry>
+        <box size="0.708 0.001 0.345"/>
+      </geometry>
+    </collision>
+    <collision name="Right_Shell">
+      <origin rpy="0 0 0" xyz="0.345 -0.177 0"/>
+      <geometry>
+        <box size="0.708 0.001 0.345"/>
+      </geometry>
+    </collision>
+    <collision name="Top_Shell">
+      <origin rpy="0 0 0" xyz="0.345 0 0.177"/>
+      <geometry>
+        <box size="0.708 0.345 0.001"/>
+      </geometry>
+    </collision>
+    <collision name="Front_Shell">
+      <origin rpy="0 0 0" xyz="0.345 0 -0.177"/>
+      <geometry>
+        <box size="0.708 0.345 0.001"/>
+      </geometry>
+    </collision>
   </link>
   <gazebo>
     <plugin filename="gz-sim-hydrodynamics-system" name="gz::sim::systems::Hydrodynamics">
       <link_name>base_link</link_name>
-      <xDotU>-2</xDotU>
-      <yDotV>-5</yDotV>
-      <zDotW>-5</zDotW>
-      <kDotP>-0.1</kDotP>
-      <mDotQ>-1</mDotQ>
-      <nDotR>-1</nDotR>
       <xUabsU>-25</xUabsU>
       <xU>-50</xU>
@@ -52,17 +83,17 @@
       <zWabsW>-5</zWabsW>
       <zW>-50</zW>
-      <kPabsP>-5</kPabsP>
-      <kP>-10</kP>
-      <mQabsQ>-5</mQabsQ>
-      <mQ>-10</mQ>
-      <nRabsR>-5</nRabsR>
-      <nR>-10</nR>
+      <kPabsP>-650</kPabsP>
+      <kP>-650</kP>
+      <mQabsQ>-750</mQabsQ>
+      <mQ>-750</mQ>
+      <nRabsR>-750</nRabsR>
+      <nR>-750</nR>
     </plugin>
   </gazebo>
   <!-- Cameras -->
-  <xacro:mil_camera name="front_cam" parent="base_link" xyz="-0.32 -0.014274 -0.050" rpy="0 0 3.14159"/>
-  <xacro:mil_camera name="down_cam" parent="base_link" xyz="-0.15222 0.027913 -0.22" rpy="0 1.57 0"/>
+  <xacro:mil_camera name="front_cam" parent="base_link" xyz="0.78 -0.014274 -0.050" rpy="0 0 0"/>
+  <xacro:mil_camera name="down_cam" parent="base_link" xyz="0.45222 0.027913 -0.22" rpy="0 1.57 0"/>
   <!-- DVL Sensor -->
-  <xacro:mil_dvl_sensor name="dvl_sensor" parent="base_link" xyz="0.21236 0.00254 -0.10233" rpy="0 0 0"/>
+  <xacro:mil_dvl_sensor name="dvl_sensor" parent="base_link" xyz="0.41236 0.00254 -0.10233" rpy="0 0 0"/>
   <!-- IMU, Magnetometer -->
   <xacro:mil_imu_magnetometer
@@ -70,5 +101,5 @@
     namespace='/imu'
     parent="base_link"
-    xyz="0.0632 -0.164 -0.079"
+    xyz="0.3632 -0.164 -0.079"
     rpy="0 0 0"
     rate="210"
@@ -81,15 +112,14 @@
   />
   <!--Depth Sensor-->
-  <xacro:mil_depth_sensor name="depth_sensor" namespace="/depth" parent="base_link" xyz="0 0 0" rpy="0 0 0" update_rate="5" frame_id="depth_sensor_frame" noise_mean="0.0" noise_stddev="0"/>
+  <xacro:mil_depth_sensor name="depth_sensor" namespace="/depth" parent="base_link" xyz="0.3 0 0" rpy="0 0 0" update_rate="5" frame_id="depth_sensor_frame" noise_mean="0.0" noise_stddev="0"/>
   <!-- Thrusters -->
   <!-- Front/Back Left/Right Vertical/Horizontal -->
-  <!-- Orientation seem to be correct -->
-  <xacro:mil_thruster name="FLV" parent="base_link" xyz="-0.15217 -0.16474 0.010449" rpy="0 0 0"/>
-  <xacro:mil_thruster name="FRV" parent="base_link" xyz="-0.1492 0.13821 0.010449" rpy="0 0 0"/>
-  <xacro:mil_thruster name="BRV" parent="base_link" xyz="0.31117 0.13821 0.010449" rpy="0 0 0"/>
-  <xacro:mil_thruster name="BLV" parent="base_link" xyz="0.30868 -0.16621 0.010449" rpy="0 0 0"/>
-  <xacro:mil_thruster name="FLH" parent="base_link" xyz="-0.14714 -0.26409 0.038317" rpy="-1.5708 0 0.7854"/>
-  <xacro:mil_thruster name="FRH" parent="base_link" xyz="-0.147 0.2413 0.038324" rpy="1.5708 0 -0.7854"/>
-  <xacro:mil_thruster name="BRH" parent="base_link" xyz="0.32369 0.22645 0.038317" rpy="-1.5708 0 0.7854"/>
-  <xacro:mil_thruster name="BLH" parent="base_link" xyz="0.32397 -0.25204 0.038324" rpy="1.5708 0 -0.7854"/>
+  <xacro:mil_thruster name="FLV" parent="base_link" xyz="0.5715 0.14922 -0.028575" rpy="0 -1.5708 0"/>
+  <xacro:mil_thruster name="FRV" parent="base_link" xyz="0.5715 -0.14922 -0.028575" rpy="0 -1.5708 0"/>
+  <xacro:mil_thruster name="BRV" parent="base_link" xyz="0.1143 -0.14922 -0.028575" rpy="0 -1.5708 0"/>
+  <xacro:mil_thruster name="BLV" parent="base_link" xyz="0.1143 0.14922 -0.028575" rpy="0 -1.5708 0"/>
+  <xacro:mil_thruster name="FLH" parent="base_link" xyz="0.58737 0.24765 0.053975" rpy="0 0 -0.523598776"/>
+  <xacro:mil_thruster name="FRH" parent="base_link" xyz="0.58737 -0.24765 0.053975" rpy="0 0 0.523598776"/>
+  <xacro:mil_thruster name="BRH" parent="base_link" xyz="0.127 -0.24765 0.053975" rpy="0 0 -0.523598776"/>
+  <xacro:mil_thruster name="BLH" parent="base_link" xyz="0.127 0.24765 0.053975" rpy="0 0 0.523598776"/>
 </robot>

File: src/subjugator/simulation/subjugator_description/urdf/xacro/thruster.xacro (robot description, xacro)
@@ -35,9 +35,8 @@
     <!-- Thruster Direction joint -->
     <joint name="${name}_dir_joint" type="revolute">
-      <origin xyz="0 0 1" rpy="0 0 0"/>
+      <origin xyz="0 0 0" rpy="0 0 0"/>
       <parent link="${name}_link"/>
       <child link="${name}_dir_link"/>
       <limit effort="1000" lower="0.0" upper="0.548" velocity="0.5"/>
-      <axis xyz="0 0 1"/>
     </joint>
     <!-- Sensor/Plugin Info-->

Commit message: decreased sim step size and decreased sub mass

File: src/subjugator/simulation/subjugator_description/urdf/sub9.urdf.xacro (robot description, xacro)
@@ -17,5 +17,5 @@
       <origin rpy="0 0 0" xyz="0.354 0 0"/>
       <!-- Need to be properly calculated at some point -->
-      <mass value="22.5"/>
+      <mass value="20.5"/>
       <inertia ixx="2.4" ixy="0" ixz="0" iyy="2.4" iyz="0.0" izz="3.0"/>
     </inertial>

Commit message: PID tuning

File: src/subjugator/simulation/subjugator_description/urdf/sub9.urdf.xacro (robot description, xacro)
@@ -16,5 +16,5 @@
     <!-- Inertial Properties -->
     <inertial>
-      <origin rpy="0 0 0" xyz="0.354 0 0"/>
+      <origin rpy="0 0 0" xyz="0.3505 0 0"/>
       <!-- Need to be properly calculated at some point -->
       <mass value="20.5"/>
@@ -33,5 +33,5 @@
       <origin rpy="0 0 0" xyz="0.354 0 0"/>
       <geometry>
-        <sphere radius="0.1725"/>
+        <sphere radius="0.1762"/>
       </geometry>
     </collision>
@@ -82,5 +82,5 @@
       <yVabsV>-25</yVabsV>
       <yV>-50</yV>
-      <zWabsW>-5</zWabsW>
+      <zWabsW>-25</zWabsW>
       <zW>-50</zW>
       <kPabsP>-25</kPabsP>
@@ -109,5 +109,5 @@
     ay="0.015707963"
     az="0.015707963"
-    lx="0.08825985"
+    lx="0.8825985"
     ly="0.08825985"
     lz="0.08825985"

Commit message: pid tuned, got rid of imu noise, ekf tuned(specifically dvl), made the sub start lower in world so that it wouldnt bounce when sim started

File: src/subjugator/simulation/subjugator_description/urdf/sub9.urdf.xacro (robot description, xacro)
@@ -16,5 +16,5 @@
     <!-- Inertial Properties -->
     <inertial>
-      <origin rpy="0 0 0" xyz="0.3505 0 0"/>
+      <origin rpy="0 0 0" xyz="0.352 0 0"/>
       <!-- Need to be properly calculated at some point -->
       <mass value="20.5"/>
@@ -33,5 +33,5 @@
       <origin rpy="0 0 0" xyz="0.354 0 0"/>
       <geometry>
-        <sphere radius="0.1762"/>
+        <sphere radius="0.1695"/>
       </geometry>
     </collision>
@@ -78,16 +78,10 @@
     <plugin filename="gz-sim-hydrodynamics-system" name="gz::sim::systems::Hydrodynamics">
       <link_name>base_link</link_name>
-      <xUabsU>-25</xUabsU>
-      <xU>-50</xU>
-      <yVabsV>-25</yVabsV>
-      <yV>-50</yV>
-      <zWabsW>-25</zWabsW>
-      <zW>-50</zW>
-      <kPabsP>-25</kPabsP>
-      <kP>-50</kP>
-      <mQabsQ>-25</mQabsQ>
-      <mQ>-50</mQ>
-      <nRabsR>-25</nRabsR>
-      <nR>-50</nR>
+      <xU>-30</xU>   <xUabsU>-15</xUabsU>
+      <yV>-40</yV>   <yVabsV>-25</yVabsV>
+      <zW>-50</zW>   <zWabsW>-25</zWabsW>
+      <kP>-30</kP>   <kPabsP>-8</kPabsP>
+      <mQ>-35</mQ>   <mQabsQ>-10</mQabsQ>
+      <nR>-40</nR>   <nRabsR>-20</nRabsR>
     </plugin>
     <plugin filename="ThrusterBridge" name="thrusterBridge::ThrusterBridge"/>
@@ -106,10 +100,10 @@
     rpy="0 3.14159 1.570797"
     rate="210"
-    ax="0.015707963"
-    ay="0.015707963"
-    az="0.015707963"
-    lx="0.8825985"
-    ly="0.08825985"
-    lz="0.08825985"
+    ax="0.0"
+    ay="0.0"
+    az="0.0"
+    lx="0.0"
+    ly="0.0"
+    lz="0.0"
   />
   <!--Depth Sensor-->

File: src/subjugator/simulation/subjugator_description/urdf/xacro/dvl.xacro (robot description, xacro)
@@ -68,5 +68,5 @@
               <bins>10</bins>
               <noise type="gaussian">
-                <stddev>0.015</stddev>
+                <stddev>0.0</stddev>
               </noise>
               <visualize>true</visualize>
@@ -75,5 +75,5 @@
               <when>best</when>
               <noise type="gaussian">
-                <stddev>0.005</stddev>
+                <stddev>0.0</stddev>
               </noise>
               <visualize>true</visualize>

Commit message: Testing oct 13 (#303)
* adds new frame that moves center of sub closer to center of rotation

* new front cam driver

---------

Co-authored-by: Joseph Handsome <nottellingu@gmail.com>
Co-authored-by: Joseph Handsome <jgoodman1@ufl.edu>

File: src/subjugator/simulation/subjugator_description/urdf/sub9.urdf.xacro (robot description, xacro)
@@ -92,4 +92,11 @@
     </plugin>
   </gazebo>
+  <!-- Define a frame at the actual center of rotation -->
+  <link name="localization_center"/>
+  <joint name="base_to_localization" type="fixed">
+    <parent link="localization_center"/>
+    <child link="base_link"/>
+    <origin xyz="-0.354 0 0" rpy="0 0 0"/>
+  </joint>
   <!-- Cameras -->
   <xacro:mil_camera name="front_cam" parent="base_link" xyz="0.78 -0.014274 -0.050" rpy="0 0 0"/>
