Commit message: Trying to add collision boxes to test optionA for picking up the object but not working :( ... I guess I at least got the arms moving cleanly

File: src/subjugator/simulation/subjugator_description/urdf/sub9.urdf (robot description, URDF)
Before this commit: robot sub9, 28 links, 27 joints
Links:
- link gripper_leftArm_link: geometry collision box ; visual mesh filename=package://subjugator_description/models/gripper_2025/grippe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
- link gripper_rightArm_link: geometry collision box ; visual mesh filename=package://subjugator_description/models/gripper_2025/grippe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

File: src/subjugator/simulation/subjugator_description/urdf/xacro/gripper.xacro (robot description, xacro)
@@ -37,5 +37,14 @@
         </geometry>
       </visual>
-      <!-- Left arm collision removed to avoid crossing/overlap issues during motion -->
+      <!-- Left fingertip collision: small rectangular box for reliable contact -->
+      <collision name="leftArm_collision">
+        <!-- positioned near the visual fingertip; adjust if needed -->
+        <origin xyz="0 0.045 0" rpy="0 0 0"/>
+        <geometry>
+          <box>
+            <size>0.1 0.1 0.1</size>
+          </box>
+        </geometry>
+      </collision>
     </link>
     <!-- Left Arm Joint -->
@@ -61,5 +70,14 @@
         </geometry>
       </visual>
-      <!-- Right arm collision removed to avoid crossing/overlap issues during motion -->
+      <!-- Right fingertip collision: small rectangular box for reliable contact -->
+      <collision name="rightArm_collision">
+        <!-- positioned near the visual fingertip; adjust if needed -->
+        <origin xyz="0 -0.045 0" rpy="0 0 0"/>
+        <geometry>
+          <box>
+            <size>0.1 0.1 0.1</size>
+          </box>
+        </geometry>
+      </collision>
     </link>
     <!-- Right Arm Joint -->

Commit message: I fixed the collision. I think its time to also re-design the gripper arm models to be like excavators rather than skeleton arms. I have witnessed it pick up a dummy box I placed once so there is potential but the physics can bug out especially with the wonky sub movement

File: src/subjugator/simulation/subjugator_description/urdf/sub9.urdf (robot description, URDF)
Before this commit: robot sub9, 28 links, 27 joints
Links:
- link gripper_leftArm_link: geometry collision mesh filename=package://subjugator_description/models/gripper_2025/grippe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 scale=1.1 1.1 1.1; visual mesh filename=package://subjugator_description/models/gripper_2025/grippe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
- link gripper_rightArm_link: geometry collision mesh filename=package://subjugator_description/models/gripper_2025/grippe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 scale=1.1 1.1 1.1; visual mesh filename=package://subjugator_description/models/gripper_2025/grippe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

File: src/subjugator/simulation/subjugator_description/urdf/xacro/gripper.xacro (robot description, xacro)
@@ -39,20 +39,8 @@
       <!-- Left fingertip collision: small rectangular box for reliable contact -->
       <collision name="leftArm_collision">
-        <!-- positioned to align with the visual finger tip (z ~ -0.3) -->
-        <origin xyz="0 0.045 -0.32" rpy="0 0 0"/>
+        <origin xyz="0 -0.025 -0.3" rpy="0 0 0"/>
         <geometry>
-          <box>
-            <size>0.02 0.04 0.06</size>
-          </box>
+          <mesh filename="package://subjugator_description/models/gripper_2025/gripper_arm.dae" scale="1.1 1.1 1.1"/>
         </geometry>
-        <!-- simple friction hint (Gazebo/ODE) -->
-        <surface>
-          <friction>
-            <ode>
-              <mu>1.0</mu>
-              <mu2>1.0</mu2>
-            </ode>
-          </friction>
-        </surface>
       </collision>
     </link>
@@ -81,20 +69,8 @@
       <!-- Right fingertip collision: small rectangular box for reliable contact -->
       <collision name="rightArm_collision">
-        <!-- positioned to align with the visual finger tip (z ~ -0.3) -->
-        <origin xyz="0 -0.045 -0.32" rpy="0 0 0"/>
+        <origin xyz="0 -0.025 -0.3" rpy="0 0 0"/>
         <geometry>
-          <box>
-            <size>0.02 0.04 0.06</size>
-          </box>
+          <mesh filename="package://subjugator_description/models/gripper_2025/gripper_arm.dae" scale="1.1 1.1 1.1"/>
         </geometry>
-        <!-- simple friction hint (Gazebo/ODE) -->
-        <surface>
-          <friction>
-            <ode>
-              <mu>1.0</mu>
-              <mu2>1.0</mu2>
-            </ode>
-          </friction>
-        </surface>
       </collision>
     </link>
@@ -117,4 +93,25 @@
       <preserveFixedJoint>true</preserveFixedJoint>
     </gazebo>
+    <!-- Gazebo-specific friction for fingertip collisions -->
+    <gazebo reference="${name}_leftArm_link">
+      <surface>
+        <friction>
+          <ode>
+            <mu>1.5</mu>
+            <mu2>1.5</mu2>
+          </ode>
+        </friction>
+      </surface>
+    </gazebo>
+    <gazebo reference="${name}_rightArm_link">
+      <surface>
+        <friction>
+          <ode>
+            <mu>1.5</mu>
+            <mu2>1.5</mu2>
+          </ode>
+        </friction>
+      </surface>
+    </gazebo>
   </xacro:macro>
 </robot>

Commit message: Ok so the gripper arms actuate and theyre not insanley walrus-tooth-like. They can hold objects but are essentially impossible to pick objects up with. Dean (my hero) helped me record a video of this that I'll add to project issue

File: src/subjugator/simulation/subjugator_description/urdf/sub9.urdf (robot description, URDF)
Before this commit: robot sub9, 28 links, 27 joints
Links:
- link gripper_link: mass 1.0 -> 0.01
Joints:
- joint gripper_leftArm_joint: origin xyz=0 0.025 0 rpy=0 0 0 -> xyz=0 0 -0.1 rpy=0 0 0
- joint gripper_rightArm_joint: origin xyz=0 -0.025 0 rpy=0 0 0 -> xyz=0 0 -0.1 rpy=0 0 0

File: src/subjugator/simulation/subjugator_description/urdf/xacro/gripper.xacro (robot description, xacro)
@@ -7,5 +7,5 @@
       <inertial>
         <origin xyz="0 0 0" rpy="0 0 0"/>
-        <mass value="1.0"/>
+        <mass value="0.01"/>
         <inertia ixx="0.01" iyy="0.01" izz="0.01" ixy="0" ixz="0" iyz="0"/>
       </inertial>
@@ -26,5 +26,5 @@
     <link name="${name}_leftArm_link">
       <inertial>
-        <origin xyz="0 0.025 0" rpy="0 0 0"/>
+        <origin xyz="0 0.03 -0.025" rpy="0 0 0"/>
         <mass value="0.1"/>
         <inertia ixx="0.001" iyy="0.001" izz="0.001" ixy="0" ixz="0" iyz="0"/>
@@ -32,5 +32,5 @@
       <!-- Left Arm Visual Link -->
       <visual name="${name}_leftArm_visual">
-        <origin xyz="0 0.025 -0.3" rpy="1.57 0 -1.57"/>
+        <origin xyz="0 0.03 -0.025" rpy="1.57 0 -1.57"/>
         <geometry>
           <mesh filename="package://subjugator_description/models/gripper_2025/gripper_arm.dae"/>
@@ -39,5 +39,5 @@
       <!-- Left fingertip collision: small rectangular box for reliable contact -->
       <collision name="leftArm_collision">
-        <origin xyz="0 -0.025 -0.3" rpy="0 0 0"/>
+        <origin xyz="0 0.03 -0.025" rpy="0 0 0"/>
         <geometry>
           <mesh filename="package://subjugator_description/models/gripper_2025/gripper_arm.dae" scale="1.1 1.1 1.1"/>
@@ -47,5 +47,5 @@
     <!-- Left Arm Joint -->
     <joint name="${name}_leftArm_joint" type="revolute">
-      <origin xyz="0 0.025 0" rpy="0 0 0"/>
+      <origin xyz="0 0 -0.1" rpy="0 0 0"/>
       <parent link="${name}_link"/>
       <child link="${name}_leftArm_link"/>
@@ -56,5 +56,5 @@
     <link name="${name}_rightArm_link">
       <inertial>
-        <origin xyz="0 -0.025 0" rpy="0 0 0"/>
+        <origin xyz="0 -0.03 -0.025" rpy="0 0 0"/>
         <mass value="0.1"/>
         <inertia ixx="0.001" iyy="0.001" izz="0.001" ixy="0" ixz="0" iyz="0"/>
@@ -62,5 +62,5 @@
       <!-- Right Arm Visual Link -->
       <visual name="${name}_rightArm_visual">
-        <origin xyz="0 -0.025 -0.3" rpy="1.57 0 1.57"/>
+        <origin xyz="0 -0.03 -0.025" rpy="1.57 0 1.57"/>
         <geometry>
           <mesh filename="package://subjugator_description/models/gripper_2025/gripper_arm.dae"/>
@@ -69,5 +69,5 @@
       <!-- Right fingertip collision: small rectangular box for reliable contact -->
       <collision name="rightArm_collision">
-        <origin xyz="0 -0.025 -0.3" rpy="0 0 0"/>
+        <origin xyz="0 -0.03 -0.025" rpy="0 0 0"/>
         <geometry>
           <mesh filename="package://subjugator_description/models/gripper_2025/gripper_arm.dae" scale="1.1 1.1 1.1"/>
@@ -77,5 +77,5 @@
     <!-- Right Arm Joint -->
     <joint name="${name}_rightArm_joint" type="revolute">
-      <origin xyz="0 -0.025 0" rpy="0 0 0"/>
+      <origin xyz="0 0 -0.1" rpy="0 0 0"/>
       <parent link="${name}_link"/>
       <child link="${name}_rightArm_link"/>
