Commit message: fixed blubjugator localization in sim

File: src/subjugator/simulation/subjugator_description/urdf/sub9_sim.urdf.xacro (robot description, xacro)
@@ -78,5 +78,5 @@
   <gazebo>
     <plugin filename="gz-sim-hydrodynamics-system" name="gz::sim::systems::Hydrodynamics">
-      <link_name>base_link</link_name>
+      <link_name>localization_center</link_name>
       <xU>-30</xU>
       <xUabsU>-15</xUabsU>
@@ -95,4 +95,16 @@
     <plugin filename="MarbleDropper" name="marble_dropper::MarbleDropper"/>
   </gazebo>
+  <link name="localization_center">
+    <inertial>
+      <mass value="0.001"/>
+      <origin xyz="0 0 0" rpy="0 0 0"/>
+      <inertia ixx="1e-6" ixy="0" ixz="0" iyy="1e-6" iyz="0" izz="1e-6"/>
+    </inertial>
+  </link>
+  <joint name="base_to_localization" type="fixed">
+    <parent link="localization_center"/>
+    <child link="base_link"/>
+    <origin xyz="-0.354 0 0" rpy="0 0 0"/>
+  </joint>
   <!-- Cameras -->
   <xacro:mil_camera name="front_cam" parent="base_link" xyz="0.78 -0.014274 -0.050" rpy="0 0 0"/>

Commit message: localization center was created to adjust what localization thought was the center of the submarine on the real submarine. This was not an issue on the simulated submarine. So only for the sim urdf file i set the position of localization_center to 0 0 0. This is because having it be the same values as it is on the real submarine created rotation issues that were not there before

File: src/subjugator/simulation/subjugator_description/urdf/sub9_sim.urdf.xacro (robot description, xacro)
@@ -105,5 +105,5 @@
     <parent link="localization_center"/>
     <child link="base_link"/>
-    <origin xyz="-0.354 0 0" rpy="0 0 0"/>
+    <origin xyz="0 0 0" rpy="0 0 0"/>
   </joint>
   <!-- Cameras -->

Commit message: fixed blubjugator localization in sim (#306)
* fixed blubjugator localization in sim

* localization center was created to adjust what localization thought was the center of the submarine on the real submarine. This was not an issue on the simulated submarine. So only for the sim urdf file i set the position of localization_center to 0 0 0. This is because having it be the same values as it is on the real submarine created rotation issues that were not there before

File: src/subjugator/simulation/subjugator_description/urdf/sub9_sim.urdf.xacro (robot description, xacro)
@@ -78,5 +78,5 @@
   <gazebo>
     <plugin filename="gz-sim-hydrodynamics-system" name="gz::sim::systems::Hydrodynamics">
-      <link_name>base_link</link_name>
+      <link_name>localization_center</link_name>
       <xU>-30</xU>
       <xUabsU>-15</xUabsU>
@@ -95,4 +95,16 @@
     <plugin filename="MarbleDropper" name="marble_dropper::MarbleDropper"/>
   </gazebo>
+  <link name="localization_center">
+    <inertial>
+      <mass value="0.001"/>
+      <origin xyz="0 0 0" rpy="0 0 0"/>
+      <inertia ixx="1e-6" ixy="0" ixz="0" iyy="1e-6" iyz="0" izz="1e-6"/>
+    </inertial>
+  </link>
+  <joint name="base_to_localization" type="fixed">
+    <parent link="localization_center"/>
+    <child link="base_link"/>
+    <origin xyz="0 0 0" rpy="0 0 0"/>
+  </joint>
   <!-- Cameras -->
   <xacro:mil_camera name="front_cam" parent="base_link" xyz="0.78 -0.014274 -0.050" rpy="0 0 0"/>

Commit message: Added second gripper arm and added that with joints to gripper.xacro

File: src/subjugator/simulation/subjugator_description/urdf/sub9_sim.urdf.xacro (robot description, xacro)
@@ -11,4 +11,5 @@
   <xacro:include filename="$(find subjugator_description)/urdf/xacro/depth.xacro"/>
   <xacro:include filename="$(find subjugator_description)/urdf/xacro/uneven_yaw.xacro"/>
+  <xacro:include filename="$(find subjugator_description)/urdf/xacro/gripper.xacro"/>
   <!-- Base Link of the Sub -->
   <link name="base_link">
@@ -120,4 +121,6 @@
   <!--Uneven Yaw Object-->
   <xacro:asym_drag_plate parent="base_link" name="asym_drag" pose_x="0.8" pose_y="0" pose_z="0" mass="0.001" yV="0" yVabsV="0"/>
+  <!-- Gripper -->
+  <xacro:mil_gripper name="mil_gripper" parent="base_link" xyz="0.375 0 -0.225" rpy="0 0 0"/>
   <!-- Thrusters -->
   <!-- Front/Back Left/Right Vertical/Horizontal -->

File: src/subjugator/simulation/subjugator_description/urdf/xacro/gripper.xacro (robot description, xacro)
@@ -2,12 +2,13 @@
 <robot xmlns:xacro="http://ros.org/wiki/xacro">
   <xacro:macro name="mil_gripper" params="name parent xyz rpy">
-    <!-- Visuals and inertial for the gripper base -->
+    <!-- Gripper Base Link -->
     <link name="${name}_link">
       <origin xyz="0 0 0" rpy="0 0 0"/>
       <inertial>
         <origin xyz="0 0 0" rpy="0 0 0"/>
-        <mass value="1"/>
+        <mass value="1.0"/>
         <inertia ixx="0.01" iyy="0.01" izz="0.01" ixy="0" ixz="0" iyz="0"/>
       </inertial>
+      <!-- Visual for base -->
       <visual name="${name}_base_visual">
         <geometry>
@@ -15,12 +16,72 @@
         </geometry>
       </visual>
-      <visual name="${name}_arm_visual">
+      <!-- Collision for base -->
+      <collision>
+        <geometry>
+          <box size="0.1 0.1 0.1"/>
+        </geometry>
+      </collision>
+    </link>
+    <!-- Left Arm Link  -->
+    <link name="${name}_armLeft_link">
+      <inertial>
+        <origin xyz="0 0.025 0" rpy="0 0 0"/>
+        <mass value="0.1"/>
+        <inertia ixx="0.001" iyy="0.001" izz="0.001" ixy="0" ixz="0" iyz="0"/>
+      </inertial>
+      <!-- Left Arm Visual Link -->
+      <visual name="${name}_armLeft_visual">
+        <origin xyz="0 0.025 -0.3" rpy="1.57 0 -1.57"/>
         <geometry>
           <mesh filename="package://subjugator_description/models/gripper_2025/gripper_arm.dae"/>
         </geometry>
       </visual>
-      <!-- Collision will be added here if needed -->
+      <!-- Left Arm Collision -->
+      <!-- <collision>
+        <origin xyz="0 0.025 -0.3" rpy="1.57 0 -1.57"/>
+        <geometry>
+          <mesh filename="package://subjugator_description/models/gripper_2025/gripper_arm.dae"/>
+        </geometry>
+      </collision> -->
     </link>
-    <!-- Fixed joint attaching gripper to parent link (pose provided by xyz/rpy params) -->
+    <!-- Left Arm Joint -->
+    <joint name="${name}_armLeft_joint" type="revolute">
+      <origin xyz="0 0.025 0" rpy="0 0 0"/>
+      <parent link="${name}_link"/>
+      <child link="${name}_armLeft_link"/>
+      <axis xyz="0 1 0"/>
+      <limit effort="1.0" velocity="1.0" lower="0.0" upper="0.5"/>
+    </joint>
+    <!-- Right Arm Link -->
+    <link name="${name}_armRight_link">
+      <inertial>
+        <origin xyz="0 -0.025 0" rpy="0 0 0"/>
+        <mass value="0.1"/>
+        <inertia ixx="0.001" iyy="0.001" izz="0.001" ixy="0" ixz="0" iyz="0"/>
+      </inertial>
+      <!-- Right Arm Visual Link -->
+      <visual name="${name}_armRight_visual">
+        <origin xyz="0 -0.025 -0.3" rpy="1.57 0 1.57"/>
+        <geometry>
+          <mesh filename="package://subjugator_description/models/gripper_2025/gripper_arm.dae"/>
+        </geometry>
+      </visual>
+      <!-- Right Arm Collision -->
+      <!-- <collision>
+        <origin xyz="0 -0.025 -0.3" rpy="1.57 0 1.57"/>
+        <geometry>
+          <mesh filename="package://subjugator_description/models/gripper_2025/gripper_arm.dae"/>
+        </geometry>
+      </collision> -->
+    </link>
+    <!-- Right Arm Joint -->
+    <joint name="${name}_armRight_joint" type="revolute">
+      <origin xyz="0 -0.025 0" rpy="0 0 0"/>
+      <parent link="${name}_link"/>
+      <child link="${name}_armRight_link"/>
+      <axis xyz="0 1 0"/>
+      <limit effort="1.0" velocity="1.0" lower="0.0" upper="0.5"/>
+    </joint>
+    <!-- Fixed Joint to Parent -->
     <joint name="${name}_joint" type="fixed">
       <origin xyz="${xyz}" rpy="${rpy}"/>
@@ -28,5 +89,4 @@
       <child link="${name}_link"/>
     </joint>
-    <!-- Ensure Gazebo does not lump away the fixed joint when spawning -->
     <gazebo reference="${name}_joint">
       <disableFixedJointLumping>true</disableFixedJointLumping>

Commit message: Gripper is visually connected to the sub with two arms

File: src/subjugator/simulation/subjugator_description/urdf/sub9_sim.urdf.xacro (robot description, xacro)
@@ -122,5 +122,5 @@
   <xacro:asym_drag_plate parent="base_link" name="asym_drag" pose_x="0.8" pose_y="0" pose_z="0" mass="0.001" yV="0" yVabsV="0"/>
   <!-- Gripper -->
-  <xacro:mil_gripper name="mil_gripper" parent="base_link" xyz="0.375 0 -0.225" rpy="0 0 0"/>
+  <xacro:gripper name="gripper" parent="base_link" xyz="0.375 0 -0.225" rpy="0 0 0"/>
   <!-- Thrusters -->
   <!-- Front/Back Left/Right Vertical/Horizontal -->

File: src/subjugator/simulation/subjugator_description/urdf/xacro/gripper.xacro (robot description, xacro)
@@ -1,5 +1,5 @@
 <?xml version="1.0"?>
 <robot xmlns:xacro="http://ros.org/wiki/xacro">
-  <xacro:macro name="mil_gripper" params="name parent xyz rpy">
+  <xacro:macro name="gripper" params="name parent xyz rpy">
     <!-- Gripper Base Link -->
     <link name="${name}_link">
@@ -24,5 +24,5 @@
     </link>
     <!-- Left Arm Link  -->
-    <link name="${name}_armLeft_link">
+    <link name="${name}_leftArm_link">
       <inertial>
         <origin xyz="0 0.025 0" rpy="0 0 0"/>
@@ -31,5 +31,5 @@
       </inertial>
       <!-- Left Arm Visual Link -->
-      <visual name="${name}_armLeft_visual">
+      <visual name="${name}_leftArm_visual">
         <origin xyz="0 0.025 -0.3" rpy="1.57 0 -1.57"/>
         <geometry>
@@ -46,13 +46,13 @@
     </link>
     <!-- Left Arm Joint -->
-    <joint name="${name}_armLeft_joint" type="revolute">
+    <joint name="${name}_leftArm_joint" type="revolute">
       <origin xyz="0 0.025 0" rpy="0 0 0"/>
       <parent link="${name}_link"/>
-      <child link="${name}_armLeft_link"/>
+      <child link="${name}_leftArm_link"/>
       <axis xyz="0 1 0"/>
       <limit effort="1.0" velocity="1.0" lower="0.0" upper="0.5"/>
     </joint>
     <!-- Right Arm Link -->
-    <link name="${name}_armRight_link">
+    <link name="${name}_rightArm_link">
       <inertial>
         <origin xyz="0 -0.025 0" rpy="0 0 0"/>
@@ -61,5 +61,5 @@
       </inertial>
       <!-- Right Arm Visual Link -->
-      <visual name="${name}_armRight_visual">
+      <visual name="${name}_rightArm_visual">
         <origin xyz="0 -0.025 -0.3" rpy="1.57 0 1.57"/>
         <geometry>
@@ -76,8 +76,8 @@
     </link>
     <!-- Right Arm Joint -->
-    <joint name="${name}_armRight_joint" type="revolute">
+    <joint name="${name}_rightArm_joint" type="revolute">
       <origin xyz="0 -0.025 0" rpy="0 0 0"/>
       <parent link="${name}_link"/>
-      <child link="${name}_armRight_link"/>
+      <child link="${name}_rightArm_link"/>
       <axis xyz="0 1 0"/>
       <limit effort="1.0" velocity="1.0" lower="0.0" upper="0.5"/>

Commit message: Added second buoyancy object

File: src/subjugator/simulation/subjugator_description/urdf/sub9_sim.urdf.xacro (robot description, xacro)
@@ -30,7 +30,14 @@
     </visual>
     <!-- Collision Data -->
-    <collision name="buoyancy_collision">
+    <collision name="buoyancy_collision_1">
       <!-- This collision is for calculating the buoyant forces-->
-      <origin rpy="0 0 0" xyz="0.354 0 0"/>
+      <origin rpy="0 0 0" xyz="0 0 0"/>
+      <geometry>
+        <sphere radius="0.01"/>
+      </geometry>
+    </collision>
+    <!-- Second buoyancy collision. Adds an additional buoyant object-->
+    <collision name="buoyancy_collision_2">
+      <origin rpy="0 0 0" xyz="0.708 0 0"/>
       <geometry>
         <sphere radius="0.1695"/>

Commit message: Added visual texture

File: src/subjugator/simulation/subjugator_description/urdf/sub9_sim.urdf.xacro (robot description, xacro)
@@ -32,16 +32,34 @@
     <collision name="buoyancy_collision_1">
       <!-- This collision is for calculating the buoyant forces-->
+      <origin rpy="0 0 0" xyz="0.0 0 0"/>
+      <geometry>
+        <sphere radius="0.134532"/>
+      </geometry>
+    </collision>
+    <visual name="buoyancy_visual_1">
       <origin rpy="0 0 0" xyz="0 0 0"/>
       <geometry>
-        <sphere radius="0.01"/>
+        <sphere radius="0.134532"/>
       </geometry>
-    </collision>
+      <material name="orange">
+        <color rgba="1 0.6 0 0.5"/>
+      </material>
+    </visual>
     <!-- Second buoyancy collision. Adds an additional buoyant object-->
     <collision name="buoyancy_collision_2">
       <origin rpy="0 0 0" xyz="0.708 0 0"/>
       <geometry>
-        <sphere radius="0.1695"/>
+        <sphere radius="0.134532"/>
       </geometry>
     </collision>
+    <visual name="buoyancy_visual_2">
+      <origin rpy="0 0 0" xyz="0.708 0 0"/>
+      <geometry>
+        <sphere radius="0.134532"/>
+      </geometry>
+      <material name="orange">
+        <color rgba="1 0.6 0 0.5"/>
+      </material>
+    </visual>
     <!-- The following are shell collisions. They dont contrubute to buoyancy-->
     <!-- and are for collisions -->

Commit message: Added all buoyancy objects + updated total force

File: src/subjugator/simulation/subjugator_description/urdf/sub9_sim.urdf.xacro (robot description, xacro)
@@ -32,13 +32,13 @@
     <collision name="buoyancy_collision_1">
       <!-- This collision is for calculating the buoyant forces-->
-      <origin rpy="0 0 0" xyz="0.0 0 0"/>
-      <geometry>
-        <sphere radius="0.134532"/>
+      <origin rpy="0 0 0" xyz="0.0 0.128 0.15"/>
+      <geometry>
+        <sphere radius="0.1116715973224"/>
       </geometry>
     </collision>
     <visual name="buoyancy_visual_1">
-      <origin rpy="0 0 0" xyz="0 0 0"/>
-      <geometry>
-        <sphere radius="0.134532"/>
+      <origin rpy="0 0 0" xyz="0 0.128 0.15"/>
+      <geometry>
+        <sphere radius="0.1116715973224"/>
       </geometry>
       <material name="orange">
@@ -48,13 +48,73 @@
     <!-- Second buoyancy collision. Adds an additional buoyant object-->
     <collision name="buoyancy_collision_2">
-      <origin rpy="0 0 0" xyz="0.708 0 0"/>
-      <geometry>
-        <sphere radius="0.134532"/>
+      <origin rpy="0 0 0" xyz="0.708 0.128 0.15"/>
+      <geometry>
+        <sphere radius="0.1116715973224"/>
       </geometry>
     </collision>
     <visual name="buoyancy_visual_2">
-      <origin rpy="0 0 0" xyz="0.708 0 0"/>
-      <geometry>
-        <sphere radius="0.134532"/>
+      <origin rpy="0 0 0" xyz="0.708 0.128 0.15"/>
+      <geometry>
+        <sphere radius="0.1116715973224"/>
+      </geometry>
+      <material name="orange">
+        <color rgba="1 0.6 0 0.5"/>
+      </material>
+    </visual>
+    <collision name="buoyancy_collision_3">
+      <origin rpy="0 0 0" xyz="0 -.128 .15"/>
+      <geometry>
+        <sphere radius="0.1116715973224"/>
+      </geometry>
+    </collision>
+    <visual name="buoyancy_visual_3">
+      <origin rpy="0 0 0" xyz="0 -.128 .15"/>
+      <geometry>
+        <sphere radius="0.1116715973224"/>
+      </geometry>
+      <material name="orange">
+        <color rgba="1 0.6 0 0.5"/>
+      </material>
+    </visual>
+    <collision name="buoyancy_collision_4">
+      <origin rpy="0 0 0" xyz="0.708 -.128 .15"/>
+      <geometry>
+        <sphere radius="0.1116715973224"/>
+      </geometry>
+    </collision>
+    <visual name="buoyancy_visual_4">
+      <origin rpy="0 0 0" xyz="0.708 -.128 .15"/>
+      <geometry>
+        <sphere radius="0.1116715973224"/>
+      </geometry>
+      <material name="orange">
+        <color rgba="1 0.6 0 0.5"/>
+      </material>
+    </visual>
+    <collision name="buoyancy_collision_5">
+      <origin rpy="0 0 0" xyz="0.531 0 0.15"/>
+      <geometry>
+        <sphere radius="0.1116715973224"/>
+      </geometry>
+    </collision>
+    <visual name="buoyancy_visual_5">
+      <origin rpy="0 0 0" xyz="0.4425 0 0.15"/>
+      <geometry>
+        <sphere radius="0.1116715973224"/>
+      </geometry>
+      <material name="orange">
+        <color rgba="1 0.6 0 0.5"/>
+      </material>
+    </visual>
+    <collision name="buoyancy_collision_6">
+      <origin rpy="0 0 0" xyz="0.25875 0 0.15"/>
+      <geometry>
+        <sphere radius="0.1116715973224"/>
+      </geometry>
+    </collision>
+    <visual name="buoyancy_visual_6">
+      <origin rpy="0 0 0" xyz="0.25875 0 0.15"/>
+      <geometry>
+        <sphere radius="0.1116715973224"/>
       </geometry>
       <material name="orange">

Commit message: Updated Z-axis and labeled objects

File: src/subjugator/simulation/subjugator_description/urdf/sub9_sim.urdf.xacro (robot description, xacro)
@@ -30,7 +30,8 @@
     </visual>
     <!-- Collision Data -->
+    <!-- Back Left Object -->
     <collision name="buoyancy_collision_1">
       <!-- This collision is for calculating the buoyant forces-->
-      <origin rpy="0 0 0" xyz="0.0 0.128 0.15"/>
+      <origin rpy="0 0 0" xyz="0.0 0.128 -0.05"/>
       <geometry>
         <sphere radius="0.1116715973224"/>
@@ -38,15 +39,15 @@
     </collision>
     <visual name="buoyancy_visual_1">
-      <origin rpy="0 0 0" xyz="0 0.128 0.15"/>
-      <geometry>
-        <sphere radius="0.1116715973224"/>
-      </geometry>
-      <material name="orange">
-        <color rgba="1 0.6 0 0.5"/>
-      </material>
-    </visual>
-    <!-- Second buoyancy collision. Adds an additional buoyant object-->
+      <origin rpy="0 0 0" xyz="0 0.128 -0.05"/>
+      <geometry>
+        <sphere radius="0.1116715973224"/>
+      </geometry>
+      <material name="orange">
+        <color rgba="1 0.6 0 0.5"/>
+      </material>
+    </visual>
+    <!-- Front Left Object -->
     <collision name="buoyancy_collision_2">
-      <origin rpy="0 0 0" xyz="0.708 0.128 0.15"/>
+      <origin rpy="0 0 0" xyz="0.708 0.128 -0.05"/>
       <geometry>
         <sphere radius="0.1116715973224"/>
@@ -54,14 +55,15 @@
     </collision>
     <visual name="buoyancy_visual_2">
-      <origin rpy="0 0 0" xyz="0.708 0.128 0.15"/>
-      <geometry>
-        <sphere radius="0.1116715973224"/>
-      </geometry>
-      <material name="orange">
-        <color rgba="1 0.6 0 0.5"/>
-      </material>
-    </visual>
+      <origin rpy="0 0 0" xyz="0.708 0.128 -0.05"/>
+      <geometry>
+        <sphere radius="0.1116715973224"/>
+      </geometry>
+      <material name="orange">
+        <color rgba="1 0.6 0 0.5"/>
+      </material>
+    </visual>
+    <!-- Back Right Object -->
     <collision name="buoyancy_collision_3">
-      <origin rpy="0 0 0" xyz="0 -.128 .15"/>
+      <origin rpy="0 0 0" xyz="0 -.128 -0.05"/>
       <geometry>
         <sphere radius="0.1116715973224"/>
@@ -69,14 +71,15 @@
     </collision>
     <visual name="buoyancy_visual_3">
-      <origin rpy="0 0 0" xyz="0 -.128 .15"/>
-      <geometry>
-        <sphere radius="0.1116715973224"/>
-      </geometry>
-      <material name="orange">
-        <color rgba="1 0.6 0 0.5"/>
-      </material>
-    </visual>
+      <origin rpy="0 0 0" xyz="0 -.128 -0.05"/>
+      <geometry>
+        <sphere radius="0.1116715973224"/>
+      </geometry>
+      <material name="orange">
+        <color rgba="1 0.6 0 0.5"/>
+      </material>
+    </visual>
+    <!-- Front Right Object -->
     <collision name="buoyancy_collision_4">
-      <origin rpy="0 0 0" xyz="0.708 -.128 .15"/>
+      <origin rpy="0 0 0" xyz="0.708 -.128 -0.05"/>
       <geometry>
         <sphere radius="0.1116715973224"/>
@@ -84,14 +87,15 @@
     </collision>
     <visual name="buoyancy_visual_4">
-      <origin rpy="0 0 0" xyz="0.708 -.128 .15"/>
-      <geometry>
-        <sphere radius="0.1116715973224"/>
-      </geometry>
-      <material name="orange">
-        <color rgba="1 0.6 0 0.5"/>
-      </material>
-    </visual>
+      <origin rpy="0 0 0" xyz="0.708 -.128 -0.05"/>
+      <geometry>
+        <sphere radius="0.1116715973224"/>
+      </geometry>
+      <material name="orange">
+        <color rgba="1 0.6 0 0.5"/>
+      </material>
+    </visual>
+    <!-- Top Front Object -->
     <collision name="buoyancy_collision_5">
-      <origin rpy="0 0 0" xyz="0.531 0 0.15"/>
+      <origin rpy="0 0 0" xyz="0.4425 0 0.15"/>
       <geometry>
         <sphere radius="0.1116715973224"/>
@@ -107,4 +111,5 @@
       </material>
     </visual>
+    <!-- Top Back Object -->
     <collision name="buoyancy_collision_6">
       <origin rpy="0 0 0" xyz="0.25875 0 0.15"/>

Commit message: Corrected shell name and increased mass to match volume displaced added by object

File: src/subjugator/simulation/subjugator_description/urdf/sub9_sim.urdf.xacro (robot description, xacro)
@@ -70,5 +70,5 @@
       </geometry>
     </collision>
-    <collision name="Front_Shell">
+    <collision name="Bottom_Shell">
       <origin rpy="0 0 0" xyz="0.345 0 -0.177"/>
       <geometry>
@@ -95,8 +95,8 @@
     <plugin filename="ThrusterBridge" name="thrusterBridge::ThrusterBridge"/>
     <plugin filename="MarbleDropper" name="marble_dropper::MarbleDropper"/>
-    <plugin filename="GripperControl" name="gripper_control::GripperControl">
+    <!-- <plugin filename="GripperControl" name="gripper_control::GripperControl">
       <left_joint_name>gripper_leftArm_joint</left_joint_name>
       <right_joint_name>gripper_rightArm_joint</right_joint_name>
-    </plugin>
+    </plugin> -->
   </gazebo>
   <link name="localization_center">
@@ -126,5 +126,5 @@
   <xacro:asym_drag_plate parent="base_link" name="asym_drag" pose_x="0.8" pose_y="0" pose_z="0" mass="0.001" yV="0" yVabsV="0"/>
   <!-- Gripper -->
-  <xacro:gripper name="gripper" parent="base_link" xyz="0.375 0 -0.225" rpy="0 0 0"/>
+  <xacro:gripper name="gripper" parent="base_link" xyz="0.354 0 -0.225" rpy="0 0 0"/>
   <!-- Thrusters -->
   <!-- Front/Back Left/Right Vertical/Horizontal -->

File: src/subjugator/simulation/subjugator_description/urdf/xacro/gripper.xacro (robot description, xacro)
@@ -7,5 +7,5 @@
       <inertial>
         <origin xyz="0 0 0" rpy="0 0 0"/>
-        <mass value="0.01"/>
+        <mass value="1.0"/>
         <inertia ixx="0.01" iyy="0.01" izz="0.01" ixy="0" ixz="0" iyz="0"/>
       </inertial>
