Commit message: Updated inertial and mass values

File: src/subjugator/simulation/subjugator_description/urdf/sub9_sim.urdf.xacro (robot description, xacro)
@@ -19,6 +19,6 @@
       <origin rpy="0 0 0" xyz="0.352 0 0"/>
       <!-- Need to be properly calculated at some point -->
-      <mass value="20.5"/>
-      <inertia ixx="2.4" ixy="0" ixz="0" iyy="2.4" iyz="0.0" izz="3.0"/>
+      <mass value="29.67"/>
+      <inertia ixx="0.8726" ixy="0.06649" ixz="-0.1350" iyy="1.980" iyz="-0.02051" izz="2.025"/>
     </inertial>
     <!-- Visual Data-->
@@ -35,5 +35,5 @@
       <origin rpy="0 0 0" xyz="0.0 0.128 -0.05"/>
       <geometry>
-        <sphere radius="0.1116715973224"/>
+        <sphere radius="0.087986820425585"/>
       </geometry>
     </collision>
@@ -41,5 +41,5 @@
       <origin rpy="0 0 0" xyz="0 0.128 -0.05"/>
       <geometry>
-        <sphere radius="0.1116715973224"/>
+        <sphere radius="0.087986820425585"/>
       </geometry>
       <material name="orange">
@@ -51,5 +51,5 @@
       <origin rpy="0 0 0" xyz="0.708 0.128 -0.05"/>
       <geometry>
-        <sphere radius="0.1116715973224"/>
+        <sphere radius="0.087986820425585"/>
       </geometry>
     </collision>
@@ -57,5 +57,5 @@
       <origin rpy="0 0 0" xyz="0.708 0.128 -0.05"/>
       <geometry>
-        <sphere radius="0.1116715973224"/>
+        <sphere radius="0.087986820425585"/>
       </geometry>
       <material name="orange">
@@ -67,5 +67,5 @@
       <origin rpy="0 0 0" xyz="0 -.128 -0.05"/>
       <geometry>
-        <sphere radius="0.1116715973224"/>
+        <sphere radius="0.087986820425585"/>
       </geometry>
     </collision>
@@ -73,5 +73,5 @@
       <origin rpy="0 0 0" xyz="0 -.128 -0.05"/>
       <geometry>
-        <sphere radius="0.1116715973224"/>
+        <sphere radius="0.087986820425585"/>
       </geometry>
       <material name="orange">
@@ -83,5 +83,5 @@
       <origin rpy="0 0 0" xyz="0.708 -.128 -0.05"/>
       <geometry>
-        <sphere radius="0.1116715973224"/>
+        <sphere radius="0.087986820425585"/>
       </geometry>
     </collision>
@@ -89,5 +89,5 @@
       <origin rpy="0 0 0" xyz="0.708 -.128 -0.05"/>
       <geometry>
-        <sphere radius="0.1116715973224"/>
+        <sphere radius="0.087986820425585"/>
       </geometry>
       <material name="orange">
@@ -99,5 +99,5 @@
       <origin rpy="0 0 0" xyz="0.4425 0 0.15"/>
       <geometry>
-        <sphere radius="0.1116715973224"/>
+        <sphere radius="0.14120533335187"/>
       </geometry>
     </collision>
@@ -105,5 +105,5 @@
       <origin rpy="0 0 0" xyz="0.4425 0 0.15"/>
       <geometry>
-        <sphere radius="0.1116715973224"/>
+        <sphere radius="0.14120533335187"/>
       </geometry>
       <material name="orange">
@@ -115,5 +115,5 @@
       <origin rpy="0 0 0" xyz="0.25875 0 0.15"/>
       <geometry>
-        <sphere radius="0.1116715973224"/>
+        <sphere radius="0.14120533335187"/>
       </geometry>
     </collision>
@@ -121,5 +121,5 @@
       <origin rpy="0 0 0" xyz="0.25875 0 0.15"/>
       <geometry>
-        <sphere radius="0.1116715973224"/>
+        <sphere radius="0.14120533335187"/>
       </geometry>
       <material name="orange">
@@ -175,6 +175,6 @@
       <zW>-50</zW>
       <zWabsW>-25</zWabsW>
-      <kP>-30</kP>
-      <kPabsP>-8</kPabsP>
+      <kP>-15</kP>
+      <kPabsP>-4</kPabsP>
       <mQ>-35</mQ>
       <mQabsQ>-10</mQabsQ>

Commit message: Add S4 grasp confirmation by scale and grasp-target config
Confirm a grasp by comparing the selected object's down-cam pixel area before
and after the lift (held object keeps its apparent size, a miss shrinks): new
RecordTargetScale / ConfirmGraspByScale leaves (detection_scale helper), wired
into the ApproachAndGrasp sequence. Adds config/grasp_targets.yaml (loaded onto
the blackboard and used as the sim graspable allowlist), documents the Servo
PWM-angle convention, and updates the GripperControl sim plugin plus world/model
plumbing. OctagonGraspMission now takes its target via a {grasp_target} port.

Sim props are still placeholders (Pink_Bin/Yellow_Bin/Yellow_Cup/Pink_Spoon),
consistent between grasp_targets.yaml and robosub_2025.world; swapping in the
real Task-5 objects is a follow-up.

File: src/subjugator/simulation/subjugator_description/urdf/sub9_sim.urdf.xacro (robot description, xacro)
@@ -1,4 +1,14 @@
 <?xml version="1.0"?>
 <robot xmlns:xacro="http://www.ros.org/wiki/xacro" name="sub9">
+  <!-- Canonical Task-5 grasp-target list, loaded once from mission_planner so the
+       GripperControl <graspable> allowlist below and the mission target labels share a
+       single source (mission_planner/config/grasp_targets.yaml). -->
+  <xacro:property name="grasp_cfg" value="${xacro.load_yaml('$(find mission_planner)/config/grasp_targets.yaml')}"/>
+  <xacro:macro name="graspables" params="names">
+    <xacro:if value="${names}">
+      <graspable>${names[0]}</graspable>
+      <xacro:graspables names="${names[1:]}"/>
+    </xacro:if>
+  </xacro:macro>
   <!-- XACRO INCLUDES -->
   <xacro:include filename="$(find subjugator_description)/urdf/xacro/fixed_link.xacro"/>
@@ -100,8 +110,5 @@
       <gripper_link_name>gripper_link</gripper_link_name>
       <attach_radius>0.25</attach_radius>
-      <graspable>Pink_Bin</graspable>
-      <graspable>Yellow_Bin</graspable>
-      <graspable>Yellow_Cup</graspable>
-      <graspable>Pink_Spoon</graspable>
+      <xacro:graspables names="${grasp_cfg['grasp_targets']}"/>
     </plugin>
   </gazebo>
