Commit message: sim: give sub9 metacentric height so it self-levels
base_link's center of gravity sat at the same point as the center of buoyancy
(both at z=0, x~0.353), so the two vertical forces had no lever arm between them
and produced no righting couple. The sub had no preferred attitude: any small
disturbance torque tilted it and nothing pushed back, leaving a steady few-degree
pitch/roll that the PID could only partly hold. That tilt rotated the down_cam
off nadir and corrupted the LockTargetXY ray-cast (orientation is the cast's
lever arm).

Lower the CoG 3 cm below the CoB to make the body a pendulum that returns to
level on its own. Place it directly under the *net* CoB x (0.354 -- the
volume-weighted centroid of all base_link buoyancy collisions, not the old
0.352): once vertical separation exists, even a 2 mm x-gap hangs the pendulum at
atan(0.002/0.03) ~= 3.8 deg of steady pitch. Aligning x zeroes that.

Validated in sim: at rest, pitch settles ~+1 deg (truth), down from ~+6 deg, and
roll ~0 -- the camera holds nadir-down without controller effort. The 3 cm
metacentric height is a starting value; larger gives stronger leveling under
motion and less sensitivity to residual x error.

File: src/subjugator/simulation/subjugator_description/urdf/sub9_sim.urdf.xacro (robot description, xacro)
@@ -28,5 +28,17 @@
     <!-- Inertial Properties -->
     <inertial>
-      <origin rpy="0 0 0" xyz="0.352 0 0"/>
+      <!-- CoG placed 3 cm directly BELOW the center of buoyancy to give the sub
+           positive metacentric height. Previously CoG and CoB were coincident
+           (both z=0) -> zero righting moment -> no passive self-leveling, so the
+           sub held a steady few-deg pitch/roll that tilted the down_cam and
+           corrupted the LockTargetXY ray-cast. A vertical CoB-above-CoG offset
+           makes it a pendulum that returns to level on its own.
+           x MUST match the net CoB x (0.354, the volume-weighted centroid of all
+           base_link buoyancy collisions: sphere+shells), not the old 0.352:
+           with GM introduced, a 2 mm x-gap between CoB and CoG hangs the pendulum
+           at atan(0.002/0.03) ~= 3.8 deg of steady pitch. Aligning x zeroes it.
+           z (-0.03) is the metacentric height; larger = stronger leveling and
+           less sensitive to residual x error. Tune against measured pitch. -->
+      <origin rpy="0 0 0" xyz="0.354 0 -0.03"/>
       <!-- Need to be properly calculated at some point -->
       <mass value="20.5"/>

Commit message: sim: raise metacentric height to 8 cm for approach-pitch stability
GM=3 cm self-levels the sub at rest (pitch ~1 deg) but under a sustained surge
the righting couple is too weak against the sim's surge disturbance torque and
pitch climbs to ~13 deg, tilting the down_cam enough to corrupt the LockTargetXY
ray-cast during the approach. Raising GM to 8 cm holds motion pitch to roughly
+/-5 deg (mostly ~3 deg) in a clean goal-step test with correct EKF anchoring.

Still a SIM PLACEHOLDER: the real GM is a measured ballast property of the
physical sub, not a tuned value. Set it to the real inclining-test figure when
available; this value only exists to stop the sim's attitude wander from
polluting perception during testing.

File: src/subjugator/simulation/subjugator_description/urdf/sub9_sim.urdf.xacro (robot description, xacro)
@@ -38,7 +38,12 @@
            with GM introduced, a 2 mm x-gap between CoB and CoG hangs the pendulum
            at atan(0.002/0.03) ~= 3.8 deg of steady pitch. Aligning x zeroes it.
-           z (-0.03) is the metacentric height; larger = stronger leveling and
-           less sensitive to residual x error. Tune against measured pitch. -->
-      <origin rpy="0 0 0" xyz="0.354 0 -0.03"/>
+           z (-0.08) is the metacentric height GM; larger = stronger leveling and
+           less sensitive to residual x error. 3 cm self-levels at REST but under
+           a sustained surge the sub still pitches ~13 deg (righting couple too
+           weak vs the sim's surge disturbance torque); 8 cm holds the approach
+           closer to level. SIM PLACEHOLDER: the real GM is a measured ballast
+           property of the physical sub, not this tuned value; set it to the real
+           inclining-test figure when available. -->
+      <origin rpy="0 0 0" xyz="0.354 0 -0.08"/>
       <!-- Need to be properly calculated at some point -->
       <mass value="20.5"/>
