Commit message: build the boat in an empty world

File: src/navigator/simulation/navigator_description/urdf/navigator.urdf.xacro (robot description, xacro)
@@ -1,17 +1,15 @@
 <?xml version="1.0"?>
 <robot name="navigator" xmlns:xacro="http://ros.org/wiki/xacro">
-  <!-- Defines the base vehicle -->
+  <!-- Include all dependent xacro files-->
   <xacro:include filename="$(find wamv_description)/urdf/wamv_base.urdf.xacro"/>
-  <!--Simulated sensors/actuators -->
-  <xacro:include filename="$(find wamv_gazebo)/urdf/components/mil_lidar.xacro"/>
-  <xacro:include filename="$(find wamv_gazebo)/urdf/components/wamv_gps.xacro"/>
-  <xacro:include filename="$(find wamv_gazebo)/urdf/components/wamv_imu.xacro"/>
-  <xacro:include filename="$(find wamv_gazebo)/urdf/components/wamv_camera.xacro"/>
-  <xacro:include filename="$(find wamv_gazebo)/urdf/components/ball_shooter.xacro"/>
-  <xacro:include filename="$(find wamv_gazebo)/urdf/components/wamv_pinger.xacro"/>
+  <xacro:include filename="$(find wamv_gazebo)/urdf/macros.xacro"/>
+  <xacro:include filename="$(find navigator_description)/urdf/components/mil_lidar.xacro"/>
+  <xacro:include filename="$(find navigator_description)/urdf/components/mil_engine.xacro"/>
+  <!-- Properties -->
   <xacro:property name="sensor_namespace" value="sensors/"/>
   <xacro:property name="camera_namespace" value="camera/"/>
   <xacro:property name="shooter_namespace" value="shooters/"/>
-  <xacro:property name="pinger_namespace" value="pingers/"/>
+  <xacro:property name="acoustic_namespace" value="pingers/"/>
+  <!-- Simulated sensors/actuators -->
   <xacro:wamv_camera name="front_left_cam" x="0.97" y="0.1" P="${radians(12)}"/>
   <xacro:wamv_camera name="front_right_cam" x="0.97" y="-0.1" P="${radians(12)}"/>
@@ -20,7 +18,6 @@
   <xacro:wamv_imu name="imu_wamv" x="0.24" y="0.17" z="1.5"/>
   <xacro:wamv_ball_shooter name="ball_shooter" x="0.54" y="0.3" z="1.3" pitch="-0.8" yaw="0.1"/>
-  <xacro:wamv_pinger name="hydrophones" position="1 0 -1"/>
+  <xacro:wamv_pinger pinger_name="hydrophones" sensor_name="hydrophones" position="1 0 -1"/>
   <!-- Add 4 thrusters -->
-  <xacro:include filename="$(find wamv_description)/urdf/thrusters/mil_engine.xacro"/>
   <xacro:property name="thruster_namespace" value="thrusters/"/>
   <!-- === engine === -->
@@ -29,9 +26,9 @@
   <xacro:mil_engine prefix="FL" position="1.46 0.54 0.49675" orientation="0.0 0.0 -0.785398" mech_reduction="1.35"/>
   <xacro:mil_engine prefix="FR" position="1.46 -0.54 0.49657" orientation="0.0 0.0 0.785398" mech_reduction="1.35"/>
-  <gazebo>
-    <plugin name="wamv_gazebo_thrust" filename="libusv_gazebo_thrust_plugin.so">
+  <!-- <gazebo>
+    <plugin filename="gz-sim-thruster-system" name="gz::sim::systems::Thruster">
       <cmdTimeout>1.0</cmdTimeout>
       <robotNamespace>${namespace}</robotNamespace>
-      <xacro:include filename="$(find wamv_gazebo)/urdf/thruster_layouts/mil_gazebo_thruster_config.xacro"/>
+      <xacro:include filename="$(find navigator_description)/urdf/thruster_layouts/mil_gazebo_thruster_config.xacro"/>
       <xacro:mil_gazebo_thruster_config name="BL"/>
       <xacro:mil_gazebo_thruster_config name="BR"/>
@@ -39,7 +36,6 @@
       <xacro:mil_gazebo_thruster_config name="FR"/>
     </plugin>
-  </gazebo>
+  </gazebo> -->
   <!-- Attach hydrodynamics plugin -->
-  <xacro:include filename="$(find wamv_gazebo)/urdf/macros.xacro"/>
   <xacro:usv_dynamics_gazebo name="wamv_dynamics_plugin"/>
   <!-- Attach wind plugin -->
