Commit message: bridge gz message to ros2, fix frame issues of sensors and baselink

File: src/navigator/simulation/navigator_description/urdf/components/mil_engine.xacro (robot description, xacro)
@@ -69,4 +69,11 @@
       </joint>
     </transmission>
+    <gazebo>
+      <plugin filename="gz-sim-thruster-system" name="gz::sim::systems::Thruster">
+        <namespace>${namespace}</namespace>
+        <joint_name>${prefix}_engine_propeller_joint</joint_name>
+        <topic>${thruster_namespace}${prefix}_thrust_cmd</topic>
+      </plugin>
+    </gazebo>
   </xacro:macro>
 </robot>

File: src/navigator/simulation/navigator_description/urdf/navigator.urdf.xacro (robot description, xacro)
@@ -8,13 +8,15 @@
   <!-- Properties -->
   <xacro:property name="sensor_namespace" value="sensors/"/>
-  <xacro:property name="camera_namespace" value="camera/"/>
+  <!-- <xacro:property name="camera_namespace" value="camera/"/> -->
   <xacro:property name="shooter_namespace" value="shooters/"/>
   <xacro:property name="acoustic_namespace" value="pingers/"/>
+  <!-- <xacro:property name="namespace" value="/navigator"/> -->
   <!-- Simulated sensors/actuators -->
+  <!-- <xacro:main_collisions prefix="navigator"/> -->
   <xacro:wamv_camera name="front_left_cam" x="0.97" y="0.1" P="${radians(12)}"/>
   <xacro:wamv_camera name="front_right_cam" x="0.97" y="-0.1" P="${radians(12)}"/>
   <xacro:mil_lidar name="velodyne" x="0.774" y="0" z="2.0" type="16_beam" P="${radians(15)}"/>
   <xacro:wamv_gps name="ins" x="0.24" y="0.17" z="1.5"/>
-  <xacro:wamv_imu name="imu_wamv" x="0.24" y="0.17" z="1.5"/>
+  <xacro:wamv_imu name="imu" x="0.24" y="0.17" z="1.5"/>
   <xacro:wamv_ball_shooter name="ball_shooter" x="0.54" y="0.3" z="1.3" pitch="-0.8" yaw="0.1"/>
   <xacro:wamv_pinger pinger_name="hydrophones" sensor_name="hydrophones" position="1 0 -1"/>
@@ -26,15 +28,4 @@
   <xacro:mil_engine prefix="FL" position="1.46 0.54 0.49675" orientation="0.0 0.0 -0.785398" mech_reduction="1.35"/>
   <xacro:mil_engine prefix="FR" position="1.46 -0.54 0.49657" orientation="0.0 0.0 0.785398" mech_reduction="1.35"/>
-  <!-- <gazebo>
-    <plugin filename="gz-sim-thruster-system" name="gz::sim::systems::Thruster">
-      <cmdTimeout>1.0</cmdTimeout>
-      <robotNamespace>${namespace}</robotNamespace>
-      <xacro:include filename="$(find navigator_description)/urdf/thruster_layouts/mil_gazebo_thruster_config.xacro"/>
-      <xacro:mil_gazebo_thruster_config name="BL"/>
-      <xacro:mil_gazebo_thruster_config name="BR"/>
-      <xacro:mil_gazebo_thruster_config name="FL"/>
-      <xacro:mil_gazebo_thruster_config name="FR"/>
-    </plugin>
-  </gazebo> -->
   <!-- Attach hydrodynamics plugin -->
   <xacro:usv_dynamics_gazebo name="wamv_dynamics_plugin"/>

File: src/navigator/simulation/navigator_description/urdf/thruster_layouts/mil_gazebo_thruster_config.xacro (robot description, xacro)
@@ -4,16 +4,6 @@
     <thruster>
       <!-- Required Parameters -->
-      <linkName>${name}_propeller_link</linkName>
       <joint_name>${name}_engine_propeller_joint</joint_name>
-      <engineJointName>${name}_chasis_engine_joint</engineJointName>
-      <cmdTopic>${thruster_namespace}${name}_thrust_cmd</cmdTopic>
-      <angleTopic>${thruster_namespace}${name}_thrust_angle</angleTopic>
-      <enableAngle>${enable_angle}</enableAngle>
-      <!-- Optional Parameters -->
-      <mappingType>1</mappingType>
-      <maxCmd>1.0</maxCmd>
-      <maxForceFwd>250.0</maxForceFwd>
-      <maxForceRev>-100.0</maxForceRev>
-      <maxAngle>${pi/2}</maxAngle>
+      <topic>${thruster_namespace}${name}_thrust_cmd</topic>
     </thruster>
   </xacro:macro>

Commit message: use model name as namespace in the xacro file

File: src/navigator/simulation/navigator_description/urdf/components/mil_engine.xacro (robot description, xacro)
@@ -71,7 +71,11 @@
     <gazebo>
       <plugin filename="gz-sim-thruster-system" name="gz::sim::systems::Thruster">
-        <namespace>${namespace}</namespace>
         <joint_name>${prefix}_engine_propeller_joint</joint_name>
-        <topic>${thruster_namespace}${prefix}/thrust</topic>
+        <topic>${thruster_namespace}/${prefix}/thrust</topic>
+      </plugin>
+      <plugin filename="gz-sim-joint-position-controller-system" name="gz::sim::systems::JointPositionController">
+        <joint_name>${prefix}_chasis_engine_joint</joint_name>
+        <topic>${namespace}/${thruster_namespace}/${prefix}/pos</topic>
+        <p_gain>1</p_gain>
       </plugin>
     </gazebo>

File: src/navigator/simulation/navigator_description/urdf/navigator.urdf.xacro (robot description, xacro)
@@ -8,8 +8,7 @@
   <!-- Properties -->
   <xacro:property name="sensor_namespace" value="sensors/"/>
-  <!-- <xacro:property name="camera_namespace" value="camera/"/> -->
+  <xacro:property name="camera_namespace" value="camera/"/>
   <xacro:property name="shooter_namespace" value="shooters/"/>
   <xacro:property name="acoustic_namespace" value="pingers/"/>
-  <!-- <xacro:property name="namespace" value="/navigator"/> -->
   <!-- Simulated sensors/actuators -->
   <!-- <xacro:main_collisions prefix="navigator"/> -->
@@ -22,5 +21,5 @@
   <xacro:wamv_pinger pinger_name="hydrophones" sensor_name="hydrophones" position="1 0 -1"/>
   <!-- Add 4 thrusters -->
-  <xacro:property name="thruster_namespace" value="thrusters/"/>
+  <xacro:property name="thruster_namespace" value="thrusters"/>
   <!-- === engine === -->
   <xacro:mil_engine prefix="BL" position="-1.9304 1.1 0.318237" orientation="0.0 0.0 0.785398" mech_reduction="1.35"/>

Commit message: Revert "use model name as namespace in the xacro file"
This reverts commit 42f6af1f330db151a677bc73734e78bd7d8f9a29.

File: src/navigator/simulation/navigator_description/urdf/components/mil_engine.xacro (robot description, xacro)
@@ -71,11 +71,7 @@
     <gazebo>
       <plugin filename="gz-sim-thruster-system" name="gz::sim::systems::Thruster">
+        <namespace>${namespace}</namespace>
         <joint_name>${prefix}_engine_propeller_joint</joint_name>
-        <topic>${thruster_namespace}/${prefix}/thrust</topic>
-      </plugin>
-      <plugin filename="gz-sim-joint-position-controller-system" name="gz::sim::systems::JointPositionController">
-        <joint_name>${prefix}_chasis_engine_joint</joint_name>
-        <topic>${namespace}/${thruster_namespace}/${prefix}/pos</topic>
-        <p_gain>1</p_gain>
+        <topic>${thruster_namespace}${prefix}/thrust</topic>
       </plugin>
     </gazebo>

File: src/navigator/simulation/navigator_description/urdf/navigator.urdf.xacro (robot description, xacro)
@@ -8,7 +8,8 @@
   <!-- Properties -->
   <xacro:property name="sensor_namespace" value="sensors/"/>
-  <xacro:property name="camera_namespace" value="camera/"/>
+  <!-- <xacro:property name="camera_namespace" value="camera/"/> -->
   <xacro:property name="shooter_namespace" value="shooters/"/>
   <xacro:property name="acoustic_namespace" value="pingers/"/>
+  <!-- <xacro:property name="namespace" value="/navigator"/> -->
   <!-- Simulated sensors/actuators -->
   <!-- <xacro:main_collisions prefix="navigator"/> -->
@@ -21,5 +22,5 @@
   <xacro:wamv_pinger pinger_name="hydrophones" sensor_name="hydrophones" position="1 0 -1"/>
   <!-- Add 4 thrusters -->
-  <xacro:property name="thruster_namespace" value="thrusters"/>
+  <xacro:property name="thruster_namespace" value="thrusters/"/>
   <!-- === engine === -->
   <xacro:mil_engine prefix="BL" position="-1.9304 1.1 0.318237" orientation="0.0 0.0 0.785398" mech_reduction="1.35"/>

Commit message: bridge thruster thrust and joint position

File: src/navigator/simulation/navigator_description/urdf/components/mil_engine.xacro (robot description, xacro)
@@ -71,7 +71,10 @@
     <gazebo>
       <plugin filename="gz-sim-thruster-system" name="gz::sim::systems::Thruster">
-        <namespace>${namespace}</namespace>
         <joint_name>${prefix}_engine_propeller_joint</joint_name>
         <topic>${thruster_namespace}${prefix}/thrust</topic>
+      </plugin>
+      <plugin filename="gz-sim-joint-position-controller-system" name="gz::sim::systems::JointPositionController">
+        <joint_name>${prefix}_chasis_engine_joint</joint_name>
+        <topic>${model_name}/${thruster_namespace}${prefix}/pos</topic>
       </plugin>
     </gazebo>

File: src/navigator/simulation/navigator_description/urdf/navigator.urdf.xacro (robot description, xacro)
@@ -1,4 +1,5 @@
 <?xml version="1.0"?>
 <robot name="navigator" xmlns:xacro="http://ros.org/wiki/xacro">
+  <xacro:arg name="model_name" default="navigator"/>
   <!-- Include all dependent xacro files-->
   <xacro:include filename="$(find wamv_description)/urdf/wamv_base.urdf.xacro"/>
@@ -8,8 +9,7 @@
   <!-- Properties -->
   <xacro:property name="sensor_namespace" value="sensors/"/>
-  <!-- <xacro:property name="camera_namespace" value="camera/"/> -->
   <xacro:property name="shooter_namespace" value="shooters/"/>
   <xacro:property name="acoustic_namespace" value="pingers/"/>
-  <!-- <xacro:property name="namespace" value="/navigator"/> -->
+  <xacro:property name="model_name" value="$(arg model_name)"/>
   <!-- Simulated sensors/actuators -->
   <!-- <xacro:main_collisions prefix="navigator"/> -->

Commit message: use new file hierarchy for mil thrusters

File: src/navigator/simulation/navigator_description/urdf/components/mil_engine.xacro (robot description, xacro)
@@ -69,14 +69,4 @@
       </joint>
     </transmission>
-    <gazebo>
-      <plugin filename="gz-sim-thruster-system" name="gz::sim::systems::Thruster">
-        <joint_name>${prefix}_engine_propeller_joint</joint_name>
-        <topic>${thruster_namespace}${prefix}/thrust</topic>
-      </plugin>
-      <plugin filename="gz-sim-joint-position-controller-system" name="gz::sim::systems::JointPositionController">
-        <joint_name>${prefix}_chasis_engine_joint</joint_name>
-        <topic>${model_name}/${thruster_namespace}${prefix}/pos</topic>
-      </plugin>
-    </gazebo>
   </xacro:macro>
 </robot>

File: src/navigator/simulation/navigator_description/urdf/navigator.urdf.xacro (robot description, xacro)
@@ -6,5 +6,4 @@
   <xacro:include filename="$(find wamv_gazebo)/urdf/macros.xacro"/>
   <xacro:include filename="$(find navigator_description)/urdf/components/mil_lidar.xacro"/>
-  <xacro:include filename="$(find navigator_description)/urdf/components/mil_engine.xacro"/>
   <!-- Properties -->
   <xacro:property name="sensor_namespace" value="sensors/"/>
@@ -23,9 +22,5 @@
   <!-- Add 4 thrusters -->
   <xacro:property name="thruster_namespace" value="thrusters/"/>
-  <!-- === engine === -->
-  <xacro:mil_engine prefix="BL" position="-1.9304 1.1 0.318237" orientation="0.0 0.0 0.785398" mech_reduction="1.35"/>
-  <xacro:mil_engine prefix="BR" position="-1.9304 -1.1 0.318237" orientation="0.0 0.0 -0.785398" mech_reduction="1.35"/>
-  <xacro:mil_engine prefix="FL" position="1.46 0.54 0.49675" orientation="0.0 0.0 -0.785398" mech_reduction="1.35"/>
-  <xacro:mil_engine prefix="FR" position="1.46 -0.54 0.49657" orientation="0.0 0.0 0.785398" mech_reduction="1.35"/>
+  <xacro:include filename="$(find navigator_description)/urdf/thruster_layouts/mil_thrusters.xacro"/>
   <!-- Attach hydrodynamics plugin -->
   <xacro:usv_dynamics_gazebo name="wamv_dynamics_plugin"/>

File: src/navigator/simulation/navigator_description/urdf/thruster_layouts/mil_gazebo_thruster_config.xacro (robot description, xacro)
@@ -1,10 +1,15 @@
 <?xml version="1.0"?>
 <plugin xmlns:xacro="http://ros.org/wiki/xacro">
-  <xacro:macro name="mil_gazebo_thruster_config" params="name enable_angle:=true">
-    <thruster>
-      <!-- Required Parameters -->
-      <joint_name>${name}_engine_propeller_joint</joint_name>
-      <topic>${thruster_namespace}${name}_thrust_cmd</topic>
-    </thruster>
+  <xacro:macro name="mil_gazebo_thruster_config" params="prefix">
+    <gazebo>
+      <plugin filename="gz-sim-thruster-system" name="gz::sim::systems::Thruster">
+        <joint_name>${prefix}_engine_propeller_joint</joint_name>
+        <topic>${thruster_namespace}${prefix}/thrust</topic>
+      </plugin>
+      <plugin filename="gz-sim-joint-position-controller-system" name="gz::sim::systems::JointPositionController">
+        <joint_name>${prefix}_chasis_engine_joint</joint_name>
+        <topic>${model_name}/${thruster_namespace}${prefix}/pos</topic>
+      </plugin>
+    </gazebo>
   </xacro:macro>
 </plugin>
