Commit message: gz->ROS bridge for lidar works now

File: src/prop/simulation/prop_gazebo/urdf/components/vlp16_lidar.xacro (robot description, xacro)
@@ -48,4 +48,5 @@
       <sensor type="gpu_lidar" name="vlp16_sensor">
         <topic>lidar</topic>
+        <frame_id>laser_frame</frame_id>
         <update_rate>${update_rate}</update_rate>
         <lidar>

File: src/prop/simulation/prop_gazebo/urdf/lidar_platform.urdf.xacro (robot description, xacro)
@@ -6,26 +6,6 @@
     <static>true</static>
   </gazebo>
-  <link name="chassis">
-    <visual>
-      <origin xyz="0 0 0" rpy="0 0 0"/>
-      <geometry>
-        <box size="0.6 0.4 0.15"/>
-      </geometry>
-      <material name="chassis_material">
-        <color rgba="0.2 0.2 0.8 1.0"/>
-      </material>
-    </visual>
-    <collision>
-      <origin xyz="0 0 0" rpy="0 0 0"/>
-      <geometry>
-        <box size="0.6 0.4 0.15"/>
-      </geometry>
-    </collision>
-    <inertial>
-      <origin xyz="0 0 0" rpy="0 0 0"/>
-      <mass value="5.0"/>
-      <inertia ixx="0.1" iyy="0.1" izz="0.1" ixy="0" ixz="0" iyz="0"/>
-    </inertial>
-  </link>
-  <xacro:vlp16_lidar parent="chassis"/>
+  <!-- Bare root link, no chassis geometry/mass, just an anchor for the sensor -->
+  <link name="base_link"/>
+  <xacro:vlp16_lidar parent="base_link" xyz="0 0 0" rpy="0 0 0"/>
 </robot>
