Commit message: put lidar on boat, publish goals with plan.py, controller improvements

File: src/prop/gnc/prop_localization/urdf/prop.urdf (robot description, URDF)
Before this commit: robot prop, 3 links, 2 joints
Joints:
- joint base_to_lidar: origin xyz=0 0 0.25 rpy=0 0 0 -> xyz=0 0 0.45 rpy=0 0 0

File: src/prop/simulation/prop_gazebo/xacro/components/vlp16_lidar.xacro (robot description, xacro)
@@ -13,4 +13,7 @@
     Give each instance its own name/frame/topic when a model carries more
     than one, since <topic> is absolute rather than model-scoped.
+    collision:=false leaves the puck out of the physics. A floating hull wants
+    that: the world's graded buoyancy only understands box and sphere
+    collisions and warns once per step about anything else.
   -->
   <xacro:macro
@@ -22,4 +25,5 @@
             rpy:='0 0 0'
             topic:=lidar
+            collision:=true
             update_rate:=10
             horizontal_samples:=1875
@@ -46,12 +50,14 @@
         </material>
       </visual>
-      <collision name="${name}_collision">
-        <geometry>
-          <cylinder>
-            <radius>0.05</radius>
-            <length>0.04</length>
-          </cylinder>
-        </geometry>
-      </collision>
+      <xacro:if value="${collision}">
+        <collision name="${name}_collision">
+          <geometry>
+            <cylinder>
+              <radius>0.05</radius>
+              <length>0.04</length>
+            </cylinder>
+          </geometry>
+        </collision>
+      </xacro:if>
       <sensor name="${name}_sensor" type="gpu_lidar">
         <topic>${topic}</topic>

File: src/prop/simulation/prop_gazebo/xacro/prop.sdf.xacro (robot description, xacro)
@@ -1,5 +1,7 @@
-<?xml version="1.0" ?>
+<?xml version="1.0" encoding="UTF-8"?>
 <!--
-  The prop boat. Differential thrust from two aft thrusters, floating on the
+  The prop boat. Generated into models/prop/model.sdf at build time; edit this
+  file, not that one.
+  Differential thrust from two aft thrusters, floating on the
   water plane the world's buoyancy plugin defines at z = 0.
   Sensors are mounted where prop_localization/urdf/prop.urdf says they are, and
@@ -10,9 +12,11 @@
   the newtons you ask it for.
   Numbers that also live elsewhere:
-    45 N per thruster and 0.25 m off the centreline -> max_thrust and
-    thruster_y in prop_controller/config/controller.yaml, and the same two
-    parameters on sim_thrusters.py.
+    the M200's 55.21 N ahead / 27.56 N astern and 0.27305 m off the
+    centreline (a 0.5461 m span) -> max_force_pos, max_force_neg and thruster_y in
+    prop_controller/config/controller.yaml, and the same three on
+    sim_thrusters.py.
 -->
-<sdf version="1.9">
+<sdf version="1.9" xmlns:xacro="http://www.ros.org/wiki/xacro">
+  <xacro:include filename="components/vlp16_lidar.xacro"/>
   <model name="prop">
     <link name="base_link">
@@ -65,8 +69,9 @@
         </material>
       </visual>
-      <!-- The thrusters, drawn where they sit: aft, 0.25 m either side of the
-           centreline and level with the centre of mass. -->
+      <!-- The thrusters, drawn where they sit: aft, 0.27305 m either side of
+           the centreline and level with the centre of mass. That is a 0.5461 m
+           span inside a 0.6 m beam, so they sit close to the chines. -->
       <visual name="left_thruster_visual">
-        <pose>-0.52 0.25 -0.15 0 1.5707963 0</pose>
+        <pose>-0.52 0.27305 -0.15 0 1.5707963 0</pose>
         <geometry>
           <cylinder>
@@ -81,5 +86,5 @@
       </visual>
       <visual name="right_thruster_visual">
-        <pose>-0.52 -0.25 -0.15 0 1.5707963 0</pose>
+        <pose>-0.52 -0.27305 -0.15 0 1.5707963 0</pose>
         <geometry>
           <cylinder>
@@ -162,32 +167,29 @@
         </navsat>
       </sensor>
-      <sensor name="lidar" type="gpu_lidar">
-        <pose>0 0 0.25 0 0 0</pose>
-        <topic>lidar/scan</topic>
-        <gz_frame_id>lidar_link</gz_frame_id>
-        <update_rate>10</update_rate>
-        <always_on>1</always_on>
-        <visualize>true</visualize>
-        <lidar>
-          <scan>
-            <horizontal>
-              <samples>360</samples>
-              <resolution>1</resolution>
-              <min_angle>-3.14159</min_angle>
-              <max_angle>3.14159</max_angle>
-            </horizontal>
-          </scan>
-          <range>
-            <min>0.5</min>
-            <max>50.0</max>
-            <resolution>0.01</resolution>
-          </range>
-        </lidar>
-      </sensor>
+      <!-- The mast the lidar sits on. Visual only: the hull's buoyancy is a
+           tuned number and every collision added to this link changes it. -->
+      <visual name="mast_visual">
+        <pose>0 0 0.265 0 0 0</pose>
+        <geometry>
+          <cylinder>
+            <length>0.33</length>
+            <radius>0.03</radius>
+          </cylinder>
+        </geometry>
+        <material>
+          <ambient>0.3 0.3 0.33 1</ambient>
+          <diffuse>0.3 0.3 0.33 1</diffuse>
+        </material>
+      </visual>
     </link>
+    <!-- The lidar, on top of the mast and clear of the hull, looking out over
+         the water. lidar_link and this height are also in
+         prop_localization/urdf/prop.urdf; keep the two in step. -->
+    <xacro:vlp16_lidar parent="base_link" name="lidar" frame="lidar_link" xyz="0 0 0.45" rpy="0 0 0" topic="lidar/scan" collision="false"/>
     <plugin filename="PropThrusters" name="prop_gazebo::PropThrusters">
       <link_name>base_link</link_name>
-      <thruster_y>0.25</thruster_y>
-      <max_thrust>45.0</max_thrust>
+      <thruster_y>0.27305</thruster_y>
+      <max_force_pos>55.21</max_force_pos>
+      <max_force_neg>27.56</max_force_neg>
       <topic_left>/prop/thrust/left</topic_left>
       <topic_right>/prop/thrust/right</topic_right>
@@ -196,8 +198,5 @@
          forwards far more easily than sideways, which is what makes it steer
          like a boat instead of a hovercraft. -->
-    <plugin
-      filename="gz-sim-hydrodynamics-system"
-      name="gz::sim::systems::Hydrodynamics"
-    >
+    <plugin filename="gz-sim-hydrodynamics-system" name="gz::sim::systems::Hydrodynamics">
       <link_name>base_link</link_name>
       <xU>-8.0</xU>
@@ -218,8 +217,5 @@
     <!-- Noise free pose and velocity, for scoring a run against the estimate.
          Nothing in the stack is allowed to subscribe to this. -->
-    <plugin
-      filename="gz-sim-odometry-publisher-system"
-      name="gz::sim::systems::OdometryPublisher"
-    >
+    <plugin filename="gz-sim-odometry-publisher-system" name="gz::sim::systems::OdometryPublisher">
       <odom_frame>map</odom_frame>
       <robot_base_frame>base_link</robot_base_frame>

Commit message: Started fusion between cam and lidar

File: src/prop/gnc/prop_localization/urdf/prop.urdf (robot description, URDF)
Before this commit: robot prop, 3 links, 2 joints
Links:
- added link camera_link
- added link camera_optical_frame
Joints:
- added joint base_to_camera: type fixed, parent base_link, child camera_link, origin xyz=0 0 0.5 rpy=0 0 0
- added joint camera_to_optical: type fixed, parent camera_link, child camera_optical_frame, origin xyz=0 0 0 rpy=-1.5707963267948966 0 -1.5707963267948966
